File: src/kicad/mp3player.kicad_sch (KiCad schematic)
At the start: 0 parts

Commit message: new day + schematic updates
Other:
- sheet power ports: added USB_D+, USB_D-; removed none
- sheet processing ports: added USB_D+, USB_D-; removed none
Changed lines of the file:
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@@
 	(generator "eeschema")
 	(generator_version "10.0")
-	(paper "A4")
+	(paper "A5")
+	(wire
+		(pts
+			(xy 50.165 52.705) (xy 50.165 47.625)
+		)
+		(stroke
+			(width 0)
+			(type default)
+		)
+	)
+	(wire
+		(pts
+			(xy 52.705 53.34) (xy 52.705 47.625)
+		)
+		(stroke
+			(width 0)
+			(type default)
+		)
+	)
+	(wire
+		(pts
+			(xy 52.07 53.34) (xy 52.07 59.055)
+		)
+		(stroke
+			(width 0)
+			(type default)
+		)
+	)
+	(wire
+		(pts
+			(xy 49.53 59.055) (xy 49.53 52.705)
+		)
+		(stroke
+			(width 0)
+			(type default)
+		)
+	)
+	(wire
+		(pts
+			(xy 49.53 52.705) (xy 50.165 52.705)
+		)
+		(stroke
+			(width 0)
+			(type default)
+		)
+	)
+	(wire
+		(pts
+			(xy 52.705 53.34) (xy 52.07 53.34)
+		)
+		(stroke
+			(width 0)
+			(type default)
+		)
+	)
 	(sheet
 		(at 100.33 31.115)
@@
 	)
 	(sheet
-		(at 30.48 61.595)
-		(size 57.785 24.13)
+		(at 23.495 59.055)
+		(size 37.465 24.13)
 		(exclude_from_sim no)
 		(in_bom yes)
@@
 		)
 		(property "Sheetname" "power"
-			(at 30.48 60.8834 0)
+			(at 23.495 58.3434 0)
 			(show_name no)
 			(do_not_autoplace no)
@@
 		)
 		(property "Sheetfile" "power.kicad_sch"
-			(at 30.48 86.3096 0)
-			(show_name no)
-			(do_not_autoplace no)
-			(effects
-				(font
-					(size 1.27 1.27)
-				)
-				(justify left top)
+			(at 23.495 83.7696 0)
+			(show_name no)
+			(do_not_autoplace no)
+			(effects
+				(font
+					(size 1.27 1.27)
+				)
+				(justify left top)
+			)
+		)
+		(pin "USB_D+" input
+			(at 52.07 59.055 90)
+			(effects
+				(font
+					(size 1.27 1.27)
+				)
+				(justify right)
+			)
+		)
+		(pin "USB_D-" input
+			(at 49.53 59.055 90)
+			(effects
+				(font
+					(size 1.27 1.27)
+				)
+				(justify right)
 			)
 		)
@@
 	)
 	(sheet
-		(at 30.48 92.71)
+		(at 119.38 71.12)
 		(size 57.785 26.67)
 		(exclude_from_sim no)
@@
 		)
 		(property "Sheetname" "audio"
-			(at 30.48 91.9984 0)
+			(at 119.38 70.4084 0)
 			(show_name no)
 			(do_not_autoplace no)
@@
 		)
 		(property "Sheetfile" "audio.kicad_sch"
-			(at 30.48 119.9646 0)
+			(at 119.38 98.3746 0)
 			(show_name no)
 			(do_not_autoplace no)
@@
 	)
 	(sheet
-		(at 29.845 26.035)
-		(size 58.42 25.4)
+		(at 24.13 22.225)
+		(size 36.83 25.4)
 		(exclude_from_sim no)
 		(in_bom yes)
@@
 		)
 		(property "Sheetname" "processing"
-			(at 29.845 25.3234 0)
+			(at 23.4184 47.625 90)
 			(show_name no)
 			(do_not_autoplace no)
@@
 		)
 		(property "Sheetfile" "processing.kicad_sch"
-			(at 29.845 52.0196 0)
-			(show_name no)
-			(do_not_autoplace no)
-			(effects
-				(font
-					(size 1.27 1.27)
-				)
-				(justify left top)
-			)
-		)
+			(at 61.5446 47.625 90)
+			(show_name no)
+			(do_not_autoplace no)
+			(effects
+				(font
+					(size 1.27 1.27)
+				)
+				(justify left top)
+			)
+		)
+		(pin "USB_D+" input
+			(at 52.705 47.625 270)
+			(effects
+				(font
+					(size 1.27 1.27)
+				)
+				(justify left)
+			)
+		)
+		(pin "USB_D-" input
+			(at 50.165 47.625 270)
+			(effects
+				(font
+					(size 1.27 1.27)
+				)
+				(justify left)
+			)
+		)

Commit message: new journal entry!
Other:
- sheet audio ports: added ANALOG_LDO_EN, I2S{LRCK DIN BCK SCK}, JACK_DETECTION; removed none
- sheet power ports: added BAT_SOC_SCL, BAT_SOC_SDA; removed none
- sheet processing ports: added I2S{LRCK DIN BCK SCK}; removed none
Changed lines of the file:
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@@
 	(generator_version "10.0")
 	(paper "A5")
+	(bus
+		(pts
+			(xy 60.96 34.29) (xy 79.375 34.29)
+		)
+		(stroke
+			(width 0)
+			(type default)
+		)
+	)
 	(wire
 		(pts
-			(xy 50.165 52.705) (xy 50.165 47.625)
+			(xy 52.705 47.625) (xy 52.705 59.055)
 		)
 		(stroke
@@
 	(wire
 		(pts
-			(xy 52.705 53.34) (xy 52.705 47.625)
+			(xy 50.165 47.625) (xy 50.165 59.055)
 		)
 		(stroke
@@
 		)
 	)
-	(wire
-		(pts
-			(xy 52.07 53.34) (xy 52.07 59.055)
-		)
-		(stroke
-			(width 0)
-			(type default)
-		)
-	)
-	(wire
-		(pts
-			(xy 49.53 59.055) (xy 49.53 52.705)
-		)
-		(stroke
-			(width 0)
-			(type default)
-		)
-	)
-	(wire
-		(pts
-			(xy 49.53 52.705) (xy 50.165 52.705)
-		)
-		(stroke
-			(width 0)
-			(type default)
-		)
-	)
-	(wire
-		(pts
-			(xy 52.705 53.34) (xy 52.07 53.34)
-		)
-		(stroke
-			(width 0)
-			(type default)
-		)
-	)
-	(sheet
-		(at 100.33 31.115)
-		(size 68.58 25.4)
+	(sheet
+		(at 80.01 57.785)
+		(size 38.1 24.765)
 		(exclude_from_sim no)
 		(in_bom yes)
@@
 		)
 		(property "Sheetname" "ui"
-			(at 100.33 30.4034 0)
+			(at 80.01 57.0734 0)
 			(show_name no)
 			(do_not_autoplace no)
@@
 		)
 		(property "Sheetfile" "ui.kicad_sch"
-			(at 100.33 57.0996 0)
+			(at 80.01 83.1346 0)
 			(show_name no)
 			(do_not_autoplace no)
@@
 		)
 		(pin "USB_D+" input
-			(at 52.07 59.055 90)
+			(at 52.705 59.055 90)
 			(effects
 				(font
@@
 		)
 		(pin "USB_D-" input
-			(at 49.53 59.055 90)
+			(at 50.165 59.055 90)
+			(effects
+				(font
+					(size 1.27 1.27)
+				)
+				(justify right)
+			)
+		)
+		(pin "BAT_SOC_SCL" input
+			(at 33.02 59.055 90)
+			(effects
+				(font
+					(size 1.27 1.27)
+				)
+				(justify right)
+			)
+		)
+		(pin "BAT_SOC_SDA" input
+			(at 35.56 59.055 90)
 			(effects
 				(font
@@
 	)
 	(sheet
-		(at 119.38 71.12)
-		(size 57.785 26.67)
+		(at 79.375 22.86)
+		(size 38.1 24.765)
 		(exclude_from_sim no)
 		(in_bom yes)
@@
 		)
 		(property "Sheetname" "audio"
-			(at 119.38 70.4084 0)
+			(at 79.375 22.1484 0)
 			(show_name no)
 			(do_not_autoplace no)
@@
 		)
 		(property "Sheetfile" "audio.kicad_sch"
-			(at 119.38 98.3746 0)
-			(show_name no)
-			(do_not_autoplace no)
-			(effects
-				(font
-					(size 1.27 1.27)
-				)
-				(justify left top)
+			(at 79.375 48.2096 0)
+			(show_name no)
+			(do_not_autoplace no)
+			(effects
+				(font
+					(size 1.27 1.27)
+				)
+				(justify left top)
+			)
+		)
+		(pin "ANALOG_LDO_EN" input
+			(at 79.375 30.48 180)
+			(effects
+				(font
+					(size 1.27 1.27)
+				)
+				(justify left)
+			)
+		)
+		(pin "I2S{LRCK DIN BCK SCK}" input
+			(at 79.375 34.29 180)
+			(effects
+				(font
+					(size 1.27 1.27)
+				)
+				(justify left)
+			)
+		)
+		(pin "JACK_DETECTION" input
+			(at 79.375 40.64 180)
+			(effects
+				(font
+					(size 1.27 1.27)
+				)
+				(justify left)
 			)
 		)
@@
 		(on_board yes)
 		(dnp no)
-		(fields_autoplaced yes)
 		(stroke
 			(width 0.1524)
@@
 		)
 		(property "Sheetfile" "processing.kicad_sch"
-			(at 61.5446 47.625 90)
+			(at 24.13 19.812 0)
 			(show_name no)
 			(do_not_autoplace no)
@@
 			)
 		)
+		(pin "I2S{LRCK DIN BCK SCK}" input
+			(at 60.96 34.29 0)
+			(effects
+				(font
+					(size 1.27 1.27)
+				)
+				(justify right)
+			)
+		)

Commit message: progress + new journal entry!
Other:
- sheet power ports: added POWER_BTN_SENSE, POWER_GPIO, UNREGULATED_SYSTEM; removed none
- sheet processing ports: added ANALOG_LDO_EN, BAT_SOC_SCL, BAT_SOC_SDA, DPAD{UP DOWN LEFT RIGHT CENTER}, JACK_DETECTION, POWER_BTN_SENSE, POWER_GPIO, SCREEN_POWER, VOLUME{UP DOWN}; removed none
- sheet ui ports: added DPAD{UP DOWN LEFT RIGHT CENTER}, VOLUME{UP DOWN}; removed none

Commit message: may 28th
Other:
- sheet power ports: added CHG_PIN; removed none
- sheet processing ports: added CHG_PIN; removed none
Changed lines of the file:
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@@
 	(generator_version "10.0")
 	(paper "A5")
-	(wire
-		(pts
-			(xy 118.11 40.005) (xy 92.71 40.005)
-		)
-		(stroke
-			(width 0)
-			(type default)
-		)
-	)
-	(wire
-		(pts
-			(xy 92.71 37.465) (xy 118.11 37.465)
+	(bus
+		(pts
+			(xy 102.87 31.115) (xy 142.24 31.115)
 		)
 		(stroke
@@
 	(bus
 		(pts
-			(xy 101.6 51.435) (xy 92.71 51.435)
+			(xy 122.555 51.435) (xy 102.87 51.435)
 		)
 		(stroke
@@
 	(bus
 		(pts
-			(xy 99.06 53.975) (xy 99.06 66.04)
-		)
-		(stroke
-			(width 0)
-			(type default)
-		)
-	)
-	(bus
-		(pts
-			(xy 118.11 31.115) (xy 92.71 31.115)
-		)
-		(stroke
-			(width 0)
-			(type default)
-		)
-	)
-	(bus
-		(pts
-			(xy 101.6 63.5) (xy 101.6 51.435)
+			(xy 120.015 53.975) (xy 120.015 66.04)
+		)
+		(stroke
+			(width 0)
+			(type default)
+		)
+	)
+	(wire
+		(pts
+			(xy 102.87 37.465) (xy 142.24 37.465)
+		)
+		(stroke
+			(width 0)
+			(type default)
+		)
+	)
+	(wire
+		(pts
+			(xy 58.42 88.9) (xy 58.42 56.515)
+		)
+		(stroke
+			(width 0)
+			(type default)
+		)
+	)
+	(bus
+		(pts
+			(xy 122.555 63.5) (xy 122.555 51.435)
 		)
 		(stroke
@@
 	(bus
 		(pts
-			(xy 118.11 63.5) (xy 101.6 63.5)
+			(xy 142.24 63.5) (xy 122.555 63.5)
 		)
 		(stroke
@@
 	(bus
 		(pts
-			(xy 99.06 66.04) (xy 118.11 66.04)
+			(xy 120.015 66.04) (xy 142.24 66.04)
 		)
 		(stroke
@@
 		)
 	)
-	(bus
-		(pts
-			(xy 92.71 53.975) (xy 99.06 53.975)
+	(wire
+		(pts
+			(xy 102.87 40.005) (xy 142.24 40.005)
+		)
+		(stroke
+			(width 0)
+			(type default)
+		)
+	)
+	(bus
+		(pts
+			(xy 102.87 53.975) (xy 120.015 53.975)
 		)
 		(stroke
@@
 	)
 	(sheet
-		(at 118.11 58.42)
+		(at 142.24 58.42)
 		(size 40.005 14.605)
 		(exclude_from_sim no)
@@
 		)
 		(property "Sheetname" "ui"
-			(at 118.11 57.7084 0)
+			(at 142.24 57.7084 0)
 			(show_name no)
 			(do_not_autoplace no)
@@
 		)
 		(property "Sheetfile" "ui.kicad_sch"
-			(at 118.11 73.6096 0)
+			(at 142.24 73.6096 0)
 			(show_name no)
 			(do_not_autoplace no)
@@
 		)
 		(pin "DPAD{UP DOWN LEFT RIGHT CENTER}" input
-			(at 118.11 63.5 180)
+			(at 142.24 63.5 180)
 			(effects
 				(font
@@
 		)
 		(pin "VOLUME{UP DOWN}" input
-			(at 118.11 66.04 180)
+			(at 142.24 66.04 180)
 			(effects
 				(font
@@
 			)
 		)
+		(pin "CHG_PIN" input
+			(at 58.42 88.9 90)
+			(effects
+				(font
+					(size 1.27 1.27)
+				)
+				(justify right)
+			)
+		)
 		(instances
 			(project "mp3player"
@@
 	)
 	(sheet
-		(at 118.11 28.575)
+		(at 142.24 28.575)
 		(size 38.735 19.685)
 		(exclude_from_sim no)
@@
 		)
 		(property "Sheetname" "audio"
-			(at 118.11 27.8634 0)
+			(at 142.24 27.8634 0)
 			(show_name no)
 			(do_not_autoplace no)
@@
 		)
 		(property "Sheetfile" "audio.kicad_sch"
-			(at 118.11 48.8446 0)
+			(at 142.24 48.8446 0)
 			(show_name no)
 			(do_not_autoplace no)
@@
 		)
 		(pin "ANALOG_LDO_EN" input
-			(at 118.11 40.005 180)
+			(at 142.24 40.005 180)
 			(effects
 				(font
@@
 		)
 		(pin "I2S{LRCK DIN BCK SCK}" input
-			(at 118.11 31.115 180)
+			(at 142.24 31.115 180)
 			(effects
 				(font
@@
 		)
 		(pin "JACK_DETECTION" input
-			(at 118.11 37.465 180)
+			(at 142.24 37.465 180)
 			(effects
 				(font
@@
 	(sheet
 		(at 24.765 26.67)
-		(size 67.945 29.845)
+		(size 78.105 29.845)
 		(exclude_from_sim no)
 		(in_bom yes)
@@
 		)
 		(pin "I2S{LRCK DIN BCK SCK}" input
-			(at 92.71 31.115 0)
+			(at 102.87 31.115 0)
 			(effects
 				(font
@@
 		)
 		(pin "ANALOG_LDO_EN" input
-			(at 92.71 40.005 0)
+			(at 102.87 40.005 0)
 			(effects
 				(font
@@
 		)
 		(pin "JACK_DETECTION" input
-			(at 92.71 37.465 0)
+			(at 102.87 37.465 0)
 			(effects
 				(font
@@
 		)
 		(pin "DPAD{UP DOWN LEFT RIGHT CENTER}" input
-			(at 92.71 53.975 0)
+			(at 102.87 53.975 0)
 			(effects
 				(font
@@
 		)
 		(pin "VOLUME{UP DOWN}" input
-			(at 92.71 51.435 0)
-			(effects
-				(font
-					(size 1.27 1.27)
-				)
-				(justify right)
-			)
-		)
+			(at 102.87 51.435 0)
+			(effects
+				(font
+					(size 1.27 1.27)
+				)
+				(justify right)
+			)
+		)
+		(pin "CHG_PIN" input
+			(at 58.42 56.515 270)
+			(effects
+				(font
+					(size 1.27 1.27)
+				)
+				(justify left)
+			)
+		)

Commit message: routing + may 30th update + things
Changed lines of the file:
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@@
+		)
+	)
+	(wire
+		(pts
+			(xy 36.195 56.515) (xy 36.195 88.9)
+		)
+		(stroke
+			(width 0)
+			(type default)
 		)
 	)
 	(bus
 		(pts
-			(xy 122.555 51.435) (xy 102.87 51.435)
-		)
-		(stroke
-			(width 0)
-			(type default)
-		)
-	)
-	(wire
-		(pts
-			(xy 36.195 56.515) (xy 36.195 88.9)
+			(xy 120.015 53.975) (xy 120.015 66.04)
+		)
+		(stroke
+			(width 0)
+			(type default)
+		)
+	)
+	(wire
+		(pts
+			(xy 102.87 37.465) (xy 142.24 37.465)
 		)
 		(stroke
@@
 	(bus
 		(pts
-			(xy 120.015 53.975) (xy 120.015 66.04)
-		)
-		(stroke
-			(width 0)
-			(type default)
-		)
-	)
-	(wire
-		(pts
-			(xy 102.87 37.465) (xy 142.24 37.465)
+			(xy 102.87 53.975) (xy 120.015 53.975)
 		)
 		(stroke
@@
 	(bus
 		(pts
-			(xy 102.87 53.975) (xy 120.015 53.975)
+			(xy 102.87 51.435) (xy 122.555 51.435)
 		)
 		(stroke
@@
 		)
 		(pin "DPAD{UP DOWN LEFT RIGHT CENTER}" input
+			(at 102.87 51.435 0)
+			(effects
+				(font
+					(size 1.27 1.27)
+				)
+				(justify right)
+			)
+		)
+		(pin "VOLUME{UP DOWN}" input
 			(at 102.87 53.975 0)
 			(effects
 				(font
-					(size 1.27 1.27)
-				)
-				(justify right)
-			)
-		)
-		(pin "VOLUME{UP DOWN}" input
-			(at 102.87 51.435 0)
-			(effects
-				(font
