File: src/kicad/power.kicad_sch (KiCad schematic)
At the start: 1 part, among them J2 USB_C_Receptacle_USB2.0_16P

Commit message: new day + schematic updates
Parts:
- added C27: 0.1uf, symbol Device:C
- added C28, C30: 4.7uf, symbol Device:C
- added C29: 1uf, symbol Device:C
- added C31, C33, C37, C38: 10uf, symbol Device:C
- added C32: 100nf, symbol Device:C
- added C34, C35, C36: 22uf, symbol Device:C
- added J5: Conn_01x02, symbol Connector_Generic:Conn_01x02
- added L2: 1.5uh, symbol Device:L
- added R13, R14: 5.1k, symbol Device:R
- added R15: 1.1k, symbol Device:R
- added R16: 890, symbol Device:R
- added R17, R18, R19: 10k, symbol Device:R
- added R20: 470k, symbol Device:R
- added R21: 150k, symbol Device:R
- added U7: TPS63070RNMR, TPS63070RNMR:VREG_TPS63070RNMR, symbol project_symbols:TPS63070RNMR
- added U8: BQ24075RGT, Package_DFN_QFN:VQFN-16-1EP_3x3mm_P0.5mm_EP1.6x1.6mm, symbol Battery_Management:BQ24075RGT
- added U9: MAX17048G_T10, max:SON50P200X200X80-9N, symbol project_symbols:MAX17048G_T10
Connections:
- net GND: now reaches J2.A1 (GND), J2.A12 (GND), J2.B1 (GND), J2.B12 (GND)
- net GND: now also J2.SH (SHIELD), C27.2, C28.1, C29.1, C30.1, C31.2, C32.2, C33.2, C34.2, C35.2, C36.2, C37.2, C38.1, J5.1 (Pin_1), R13.2, R14.2, R15.1, R16.1, R17.1, R21.2, U7.10 (PGND), U7.15 (VSEL), U7.4 (GND), U7.6 (FB2), U8.14 (TMR), U8.15 (SYSOFF), U8.17 (VSS), U8.4 (~{CE}), U8.6 (EN1), U8.8 (VSS), U9.1 (CTG), U9.4 (GND), U9.6 (QSTRT), U9.9 (EP)
- net USB_VBUS: now reaches J2.A4 (VBUS), J2.A9 (VBUS), J2.B4 (VBUS), J2.B9 (VBUS)
- net USB_VBUS: now also C29.2, U8.13 (IN)
- net at J2.A5 (CC1): now also R13.1
- net USB_D+: now reaches J2.A6 (D+)
- net USB_D+: now also J2.B6 (D+)
- net USB_D-: now reaches J2.A7 (D-)
- net USB_D-: now also J2.B7 (D-)
- net at J2.B5 (CC2): now also R14.1
- new net: C32.1, U7.3 (VAUX)
- new net: R15.2, U8.12 (ILIM)
- new net: R19.2, U7.2 (PG)
- new net: R18.1, U7.1 (PS/SYNC), U7.14 (EN)
- new net: L2.1, U7.9 (L2)
- new net: L2.2, U7.11 (L1)
- new net: R16.2, U8.16 (ISET)
- new net: R17.2, U8.1 (TS)
- new net: R20.2, R21.1, U7.5 (FB)
- new net +3V3: C33.1, C34.1, C35.1, C36.1, R19.1, R20.1, U7.7_8 (VOUT)
- new net BAT_SOC_SCL: U9.7 (SCL)
- new net BAT_SOC_SDA: U9.8 (SDA)
- new net B_EN2: C30.2, C31.1, C37.1, C38.2, R18.2, U7.12_13 (VIN), U8.10 (OUT), U8.11 (OUT), U8.5 (EN2)
- new net LIPO_+: C27.1, C28.2, J5.2 (Pin_2), U8.2 (BAT), U8.3 (BAT), U9.2 (CELL), U9.3 (VDD)
- no-connect marks 0 -> 5
Other:
- note added: "BAT connector"
- note added: "battery state of charge ic"
- moved on the sheet: J2

Commit message: new journal entry!
Parts:
- added D2: D_Schottky, symbol Device:D_Schottky
- added Q1: Q_NMOS, symbol Device:Q_NMOS
- added R25, R27: 10k, symbol Device:R
- added R26: 100k, symbol Device:R
- added SW12: SW_Push, symbol Switch:SW_Push
Connections:
- net +3V3: now also U7.15 (VSEL)
- net GND: now also Q1.S, R26.1; no longer U7.15 (VSEL), U8.15 (SYSOFF)
- net LIPO_+: now also R25.1, SW12.1
- new net: Q1.D, R25.2, U8.15 (SYSOFF)
- new net: D2.2 (A), SW12.2
- new net: D2.1 (K), Q1.G, R26.2, R27.1
- new net POWER_GPIO: R27.2
Other:
- note added: "side power btn"
- moved on the sheet: C27, C28, C29, C30, C33, J5, R15, R16, R17, R18, U8, U9

Commit message: progress + new journal entry!
Parts:
- removed Q1: Q_NMOS, symbol Device:Q_NMOS
- added D3: D_Schottky, symbol Device:D_Schottky
- added Q2, Q3: BSS138, Package_TO_SOT_SMD:SOT-23, symbol Transistor_FET:BSS138
Connections:
- net GND: now also Q2.2 (S), Q3.2 (S)
- net at R25.2, U8.15 (SYSOFF): now also Q2.3 (D)
- net at D2.2 (A), SW12.2: now also D3.2 (A)
- net at D2.1 (K), R26.2, R27.1: now also Q2.1 (G)
- net B_EN2 renamed UNREGULATED_SYSTEM
- new net: D3.1 (K), Q3.1 (G)
- new net POWER_BTN_SENSE: Q3.3 (D)
Other:
- moved on the sheet: D2, J2, R13, R14, SW12

Commit message: may 28th
Parts:
- removed SW12: SW_Push, symbol Switch:SW_Push
- added R28: 10k, Resistor_SMD:R_0402_1005Metric, symbol Device:R
- added SW1: EVQPUL02K, EVQPUL02K:KEY-SMD_4P-L4.7-W3.5-P1.70-LS6.4-EH, symbol Switch:SW_Push
- R25, R27: footprint (none) -> Resistor_SMD:R_0402_1005Metric
- R26: footprint (none) -> Resistor_SMD:R_0402_1005Metric; LCSC Part (none) -> C25741
- U7: footprint TPS63070RNMR:VREG_TPS63070RNMR -> misc:VREG_TPS63070RNMR; LCSC Part (none) -> C109322
- U8: LCSC Part (none) -> C15464
- U9: footprint max:SON50P200X200X80-9N -> misc:SON50P200X200X80-9N; LCSC Part (none) -> C2682616
Connections:
- net +3V3: now also R28.1
- net LIPO_+: now also SW1.1
- net POWER_BTN_SENSE: now also R28.2
- net at D2.2 (A), D3.2 (A): now also SW1.2
- net CHG_PIN: now reaches U8.9 (~{CHG})
- no-connect marks 5 -> 4

Commit message: more components associations
Parts:
- C32: footprint (none) -> Capacitor_SMD:C_0402_1005Metric; LCSC Part (none) -> C1525
- J2: footprint (none) -> easyeda2kicad:USB-C-SMD_GT-USB-7047C; LCSC Part (none) -> C963218
- Q2, Q3: LCSC Part (none) -> C52895
- R13, R14: footprint (none) -> Resistor_SMD:R_0402_1005Metric; LCSC Part (none) -> C25905
- R15: value 1.1k -> 820; footprint (none) -> Resistor_SMD:R_0603_1608Metric; LCSC Part (none) -> C23253; Tolerance (none) -> 1%
- R16: value 890 -> 1k; footprint (none) -> Resistor_SMD:R_0402_1005Metric; LCSC Part (none) -> C11702; Tolerance (none) -> 1%
- R17, R18, R19: footprint (none) -> Resistor_SMD:R_0402_1005Metric; LCSC Part (none) -> C25744
- R20: footprint (none) -> Resistor_SMD:R_0603_1608Metric; LCSC Part (none) -> C23178
- R21: footprint (none) -> Resistor_SMD:R_0603_1608Metric; LCSC Part (none) -> C22807
- R25, R27, R28: LCSC Part (none) -> C25744
Changed lines of the file:
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@@
 			)
 		)
-		(property "Footprint" ""
+		(property "Footprint" "Capacitor_SMD:C_0402_1005Metric"
 			(at 235.9152 69.85 0)
 			(hide yes)
@@
 			)
 		)
+		(property "LCSC Part" "C1525"
+			(at 234.95 66.04 90)
+			(hide yes)
+			(show_name no)
+			(do_not_autoplace no)
+			(effects
+				(font
+					(size 1.27 1.27)
+				)
+			)
+		)
 		(pin "2"
 		)
@@
 			)
 		)
+		(property "LCSC Part" "C25744"
+			(at 87.63 124.46 0)
+			(hide yes)
+			(show_name no)
+			(do_not_autoplace no)
+			(effects
+				(font
+					(size 1.27 1.27)
+				)
+			)
+		)
 		(pin "1"
 		)
@@
 			)
 		)
-		(property "Value" "1.1k"
+		(property "Value" "820"
 			(at 77.47 157.4799 0)
 			(show_name no)
@@
 			)
 		)
-		(property "Footprint" ""
+		(property "Footprint" "Resistor_SMD:R_0603_1608Metric"
 			(at 76.708 156.21 90)
 			(hide yes)
@@
 			)
 		)
+		(property "Tolerance" "1%"
+			(at 74.93 156.21 0)
+			(hide yes)
+			(show_name no)
+			(do_not_autoplace no)
+			(effects
+				(font
+					(size 1.27 1.27)
+				)
+			)
+		)
+		(property "LCSC Part" "C23253"
+			(at 74.93 156.21 0)
+			(hide yes)
+			(show_name no)
+			(do_not_autoplace no)
+			(effects
+				(font
+					(size 1.27 1.27)
+				)
+			)
+		)
 		(pin "1"
 		)
@@
 			)
 		)
-		(property "Footprint" ""
+		(property "Footprint" "Resistor_SMD:R_0402_1005Metric"
 			(at 60.96 38.608 90)
 			(hide yes)
@@
 			)
 		)
+		(property "LCSC Part" "C25905"
+			(at 60.96 36.83 90)
+			(hide yes)
+			(show_name no)
+			(do_not_autoplace no)
+			(effects
+				(font
+					(size 1.27 1.27)
+				)
+			)
+		)
 		(pin "2"
 		)
@@
 			)
 		)
+		(property "LCSC Part" "C25744"
+			(at 38.735 88.9 90)
+			(hide yes)
+			(show_name no)
+			(do_not_autoplace no)
+			(effects
+				(font
+					(size 1.27 1.27)
+				)
+			)
+		)
 		(pin "2"
 		)
@@
 			)
 		)
-		(property "Footprint" ""
+		(property "Footprint" "easyeda2kicad:USB-C-SMD_GT-USB-7047C"
 			(at 41.91 46.99 0)
 			(hide yes)
@@
 			)
 		)
+		(property "LCSC Part" "C963218"
+			(at 38.1 46.99 0)
+			(hide yes)
+			(show_name no)
+			(do_not_autoplace no)
+			(effects
+				(font
+					(size 1.27 1.27)
+				)
+			)
+		)
 		(pin "A9"
 		)
@@
 			)
 		)
-		(property "Footprint" ""
+		(property "Footprint" "Resistor_SMD:R_0402_1005Metric"
 			(at 255.27 47.752 90)
 			(hide yes)
@@
 			)
 		)
+		(property "LCSC Part" "C25744"
+			(at 255.27 49.53 90)
+			(hide yes)
+			(show_name no)
+			(do_not_autoplace no)
+			(effects
+				(font
+					(size 1.27 1.27)
+				)
+			)
+		)
 		(pin "2"
 		)
@@
 			)
 		)
+		(property "LCSC Part" "C25744"
+			(at 74.93 120.65 90)
+			(hide yes)
+			(show_name no)
+			(do_not_autoplace no)
+			(effects
+				(font
+					(size 1.27 1.27)
+				)
+			)
+		)
 		(pin "1"
 		)
@@
 			)
 		)
-		(property "Footprint" ""
+		(property "Footprint" "Resistor_SMD:R_0402_1005Metric"
 			(at 163.068 52.07 90)
 			(hide yes)
@@
 			)
 		)
+		(property "LCSC Part" "C25744"
+			(at 161.29 52.07 0)
+			(hide yes)
+			(show_name no)
+			(do_not_autoplace no)
+			(effects
+				(font
+					(size 1.27 1.27)
+				)
+			)
+		)
 		(pin "2"
 		)
@@
 			)
 		)
-		(property "Value" "890"
+		(property "Value" "1k"
 			(at 87.63 160.0199 0)
 			(show_name no)
@@
 			)
 		)
-		(property "Footprint" ""
+		(property "Footprint" "Resistor_SMD:R_0402_1005Metric"
 			(at 86.868 158.75 90)
 			(hide yes)
@@
 			)
 		)
+		(property "Tolerance" "1%"
+			(at 85.09 158.75 0)
+			(hide yes)
+			(show_name no)
+			(do_not_autoplace no)
+			(effects
+				(font
+					(size 1.27 1.27)
+				)
+			)
+		)
+		(property "LCSC Part" "C11702"
+			(at 85.09 158.75 0)
+			(hide yes)
+			(show_name no)
+			(do_not_autoplace no)
+			(effects
+				(font
+					(size 1.27 1.27)
+				)
+			)
+		)
 		(pin "1"
 		)
@@
 			)
 		)
-		(property "Footprint" ""
+		(property "Footprint" "Resistor_SMD:R_0402_1005Metric"
 			(at 77.47 41.148 90)
 			(hide yes)
@@
 			)
 		)
+		(property "LCSC Part" "C25905"
+			(at 77.47 39.37 90)
+			(hide yes)
+			(show_name no)
+			(do_not_autoplace no)
+			(effects
+				(font
+					(size 1.27 1.27)
+				)
+			)
+		)
 		(pin "2"
 		)
@@
 			)
 		)
-		(property "Footprint" ""
+		(property "Footprint" "Resistor_SMD:R_0402_1005Metric"
 			(at 129.54 149.352 90)
 			(hide yes)
@@
 			)
 		)
+		(property "LCSC Part" "C25744"
+			(at 129.54 151.13 90)
+			(hide yes)
+			(show_name no)
+			(do_not_autoplace no)
+			(effects
+				(font
+					(size 1.27 1.27)
+				)
+			)
+		)
 		(pin "1"
 		)
@@
 			)
 		)
-		(property "Footprint" ""
+		(property "Footprint" "Resistor_SMD:R_0603_1608Metric"
 			(at 247.142 66.04 90)
 			(hide yes)
@@
 			)
 		)
+		(property "LCSC Part" "C22807"
+			(at 248.92 66.04 0)
+			(hide yes)
+			(show_name no)
+			(do_not_autoplace no)
+			(effects
+				(font
+					(size 1.27 1.27)
+				)
+			)
+		)
 		(pin "2"
 		)
@@
 			)
 		)
-		(property "Footprint" ""
+		(property "Footprint" "Resistor_SMD:R_0603_1608Metric"
 			(at 247.142 55.88 90)
 			(hide yes)
@@
 			)
 		)
+		(property "LCSC Part" "C23178"
+			(at 248.92 55.88 0)
+			(hide yes)
+			(show_name no)
+			(do_not_autoplace no)
+			(effects
+				(font
+					(size 1.27 1.27)
+				)
+			)
+		)
 		(pin "2"
 		)
@@
 			)
 		)
+		(property "LCSC Part" "C52895"
+			(at 68.58 130.81 90)
+			(hide yes)
+			(show_name no)
+			(do_not_autoplace no)
+			(effects
+				(font
+					(size 1.27 1.27)
+				)
+			)
+		)
 		(pin "1"
 		)
@@
 			(at 53.34 97.79 90)
 			(hide yes)
+			(show_name no)
+			(do_not_autoplace no)
+			(effects
+				(font
+					(size 1.27 1.27)
+				)
+			)
+		)
+		(property "LCSC Part" "C52895"
+			(at 53.34 97.79 90)
+			(hide yes)

Commit message: may 29th + files updates
Parts:
- C27: footprint (none) -> Capacitor_SMD:C_0402_1005Metric; LCSC Part (none) -> C1525
- C28, C30: footprint (none) -> Capacitor_SMD:C_0603_1608Metric; LCSC Part (none) -> C19666
- C29: footprint (none) -> Capacitor_SMD:C_0402_1005Metric; LCSC Part (none) -> C52923
- C31, C33, C37, C38: footprint (none) -> Capacitor_SMD:C_0603_1608Metric; LCSC Part (none) -> C96446
- C34, C35, C36: footprint (none) -> Capacitor_SMD:C_0603_1608Metric; LCSC Part (none) -> C59461
- D2, D3: footprint (none) -> Diode_SMD:D_SOD-123; LCSC Part (none) -> C8598
- J5: footprint (none) -> Connector_JST:JST_PH_S2B-PH-SM4-TB_1x02-1MP_P2.00mm_Horizontal; LCSC Part (none) -> C295747
- L2: footprint (none) -> Inductor_SMD:L_Sunlord_MWSA0402S; LCSC Part (none) -> C408334

Commit message: jun 1st what already noo
Parts:
- R19: value 10k -> 100k; LCSC Part C25744 -> C25741
Connections:
- net +3V3: no longer U7.15 (VSEL)
- net GND: now also U7.15 (VSEL)
Changed lines of the file:
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@@
 	)
 	(junction
-		(at 231.14 46.99)
-		(diameter 0)
-		(color 0 0 0 0)
-	)
-	(junction
 		(at 250.19 29.21)
 		(diameter 0)
@@
 	(wire
 		(pts
-			(xy 191.77 49.53) (xy 186.69 49.53)
-		)
-		(stroke
-			(width 0)
-			(type default)
-		)
-	)
-	(wire
-		(pts
 			(xy 121.92 153.67) (xy 118.11 153.67)
 		)
@@
 	(wire
 		(pts
-			(xy 231.14 46.99) (xy 242.57 46.99)
+			(xy 227.33 46.99) (xy 242.57 46.99)
 		)
 		(stroke
@@
 	(wire
 		(pts
-			(xy 186.69 34.29) (xy 231.14 34.29)
-		)
-		(stroke
-			(width 0)
-			(type default)
-		)
-	)
-	(wire
-		(pts
 			(xy 265.43 46.99) (xy 261.62 46.99)
 		)
@@
 	(wire
 		(pts
-			(xy 186.69 49.53) (xy 186.69 34.29)
-		)
-		(stroke
-			(width 0)
-			(type default)
-		)
-	)
-	(wire
-		(pts
 			(xy 248.92 60.96) (xy 248.92 62.23)
 		)
@@
 	(wire
 		(pts
-			(xy 231.14 46.99) (xy 227.33 46.99)
-		)
-		(stroke
-			(width 0)
-			(type default)
-		)
-	)
-	(wire
-		(pts
 			(xy 238.76 110.49) (xy 238.76 135.89)
 		)
@@
 	(wire
 		(pts
-			(xy 231.14 34.29) (xy 231.14 46.99)
-		)
-		(stroke
-			(width 0)
-			(type default)
-		)
-	)
-	(wire
-		(pts
 			(xy 179.07 57.15) (xy 191.77 57.15)
 		)
@@
 			)
 		)
-		(property "Value" "10k"
+		(property "Value" "100k"
 			(at 255.27 45.72 90)
 			(show_name no)
@@
 			)
 		)
-		(property "LCSC Part" "C25744"
+		(property "LCSC Part" "C25741"
 			(at 255.27 49.53 90)
 			(hide yes)
@@
 					(unit 1)
 				)
+			)
+		)
+	)
+	(symbol
+		(lib_id "power:GND")
+		(at 191.77 49.53 270)
+		(unit 1)
+		(body_style 1)
+		(exclude_from_sim no)
+		(in_bom yes)
+		(on_board yes)
+		(in_pos_files yes)
+		(dnp no)
+		(fields_autoplaced yes)
+		(property "Reference" "#PWR070"
+			(at 185.42 49.53 0)
+			(hide yes)
+			(show_name no)
+			(do_not_autoplace no)
+			(effects
+				(font
+					(size 1.27 1.27)
+				)
+			)
+		)
+		(property "Value" "GND"
+			(at 187.96 49.5299 90)
+			(show_name no)
+			(do_not_autoplace no)
+			(effects
+				(font
+					(size 1.27 1.27)
+				)
+				(justify right)
+			)
+		)
+		(property "Footprint" ""
+			(at 191.77 49.53 0)
+			(hide yes)
+			(show_name no)
+			(do_not_autoplace no)
+			(effects
+				(font
+					(size 1.27 1.27)
+				)
+			)
+		)
+		(property "Datasheet" ""
+			(at 191.77 49.53 0)
+			(hide yes)
+			(show_name no)
+			(do_not_autoplace no)
+			(effects
+				(font
+					(size 1.27 1.27)
+				)
+			)
+		)
+		(property "Description" "Power symbol creates a global label with name \"GND\" , ground"
+			(at 191.77 49.53 0)
+			(hide yes)
+			(show_name no)
+			(do_not_autoplace no)
+			(effects
+				(font
+					(size 1.27 1.27)
+				)
+			)
+		)
+		(pin "1"
+		)
+		(instances
+			(project "mp3player"
+				(path "/730d0887-0a09-4397-bcb4-2959d410b5ba/727f8b88-b598-49af-b523-8d5e77923d77"
+					(reference "#PWR070")
+					(unit 1)
+				)
