File: src/kicad/power.kicad_sch (KiCad schematic)
At the start: 36 parts, among them J2 USB_C_Receptacle_USB2.0_16P, J5 Conn_01x02, Q2 BSS138, Q3 BSS138, SW1 EVQPUL02K, U7 TPS63070RNMR, U8 BQ24075RGT, U9 MAX17048G_T10

Commit message: cad added + journal/bom update
Parts:
- C27: value 0.1uf -> 100nf
- C29: LCSC Part C52923 -> C307427
- L2: LCSC Part C408334 -> C351088
- R13, R14: LCSC Part C25905 -> C852856
- R16: LCSC Part C11702 -> C852624
- R17, R18, R25, R27, R28: LCSC Part C25744 -> C2906861
- R19, R26: LCSC Part C25741 -> C481918
- R20: LCSC Part C23178 -> C2907040
- R21: LCSC Part C22807 -> C326734
Changed lines of the file:
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@@
 			)
 		)
-		(property "LCSC Part" "C25744"
+		(property "LCSC Part" "C2906861"
 			(at 87.63 124.46 0)
 			(hide yes)
@@
 			)
 		)
-		(property "LCSC Part" "C25905"
+		(property "LCSC Part" "C852856"
 			(at 60.96 36.83 90)
 			(hide yes)
@@
 			)
 		)
-		(property "LCSC Part" "C25744"
+		(property "LCSC Part" "C2906861"
 			(at 38.735 88.9 90)
 			(hide yes)
@@
 			)
 		)
-		(property "LCSC Part" "C25741"
+		(property "LCSC Part" "C481918"
 			(at 255.27 49.53 90)
 			(hide yes)
@@
 			)
 		)
-		(property "LCSC Part" "C25744"
+		(property "LCSC Part" "C2906861"
 			(at 74.93 120.65 90)
 			(hide yes)
@@
 			)
 		)
-		(property "LCSC Part" "C52923"
+		(property "LCSC Part" "C307427"
 			(at 100.33 167.64 90)
 			(hide yes)
@@
 			)
 		)
-		(property "LCSC Part" "C25744"
+		(property "LCSC Part" "C2906861"
 			(at 161.29 52.07 0)
 			(hide yes)
@@
 			)
 		)
-		(property "LCSC Part" "C408334"
+		(property "LCSC Part" "C351088"
 			(at 180.34 66.04 0)
 			(hide yes)
@@
 			)
 		)
-		(property "Value" "0.1uf"
+		(property "Value" "100nf"
 			(at 246.38 130.8099 0)
 			(show_name no)
@@
 			)
 		)
-		(property "LCSC Part" "C25741"
+		(property "LCSC Part" "C481918"
 			(at 68.58 107.95 0)
 			(hide yes)
@@
 			)
 		)
-		(property "LCSC Part" "C11702"
+		(property "LCSC Part" "C852624"
 			(at 85.09 158.75 0)
 			(hide yes)
@@
 			)
 		)
-		(property "LCSC Part" "C25905"
+		(property "LCSC Part" "C852856"
 			(at 77.47 39.37 90)
 			(hide yes)
@@
 			)
 		)
-		(property "LCSC Part" "C25744"
+		(property "LCSC Part" "C2906861"
 			(at 129.54 151.13 90)
 			(hide yes)
@@
 			)
 		)
-		(property "LCSC Part" "C22807"
+		(property "LCSC Part" "C326734"
 			(at 248.92 66.04 0)
 			(hide yes)
@@
 			)
 		)
-		(property "LCSC Part" "C23178"
+		(property "LCSC Part" "C2907040"
 			(at 248.92 55.88 0)
 			(hide yes)
