File: src/kicad/processing.kicad_sch (KiCad schematic)
At the start: 61 parts, among them J1 SD_Card_Receptacle, J4 Conn_01x03, J6 Conn_01x42, SW11 TS-1088-AR02016, U1 ABM8-272-T3_C20625731, U11 TPS61165DRV, U12 TCA9555RTWR, U2 FSC-BT1114QI, U3 W25Q128JVE, U4 APS6404L-SQRx-ZR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

Commit message: first of june wo&
Parts:
- removed C17, C18: 100nf, Capacitor_SMD:C_0402_1005Metric, symbol Device:C
Connections:
- net DISPLAY_RESET: now also U6.9 (GPIO11)

Commit message: new dayy
Parts:
- removed J4: Conn_01x03, Connector_PinHeader_2.54mm:PinHeader_1x03_P2.54mm_Vertical, symbol Connector_Generic:Conn_01x03
- added J3: Conn_01x05, misc:test_pads, symbol Connector_Generic:Conn_01x05
- added R32, R33, R38, R48: 33, Resistor_SMD:R_0402_1005Metric, symbol Device:R
Connections:
- net +3V3: now also J3.5 (Pin_5)
- net BLE_I2S_BCLK: now also R33.2; no longer U6.4 (GPIO7)
- net BLE_I2S_DIN: now also R32.2; no longer U6.3 (GPIO6)
- net BLE_I2S_MCLK: now also R48.2; no longer U6.7 (GPIO9)
- net BLE_I2S_WS: now also R38.2; no longer U6.6 (GPIO8)
- net GND: now also J3.3 (Pin_3)
- net RP_SWCLK: now also J3.4 (Pin_4)
- net RP_SWDIO: now also J3.2 (Pin_2)
- net RUN: now reaches U6.35 (RUN)
- net RUN: now also J3.1 (Pin_1)
- new net: R32.1, U6.3 (GPIO6)
- new net: R48.1, U6.7 (GPIO9)
- new net: R33.1, U6.4 (GPIO7)
- new net: R38.1, U6.6 (GPIO8)

Commit message: new day!
Connections:
- net EXPANDER_INT: now also U6.57 (GPIO46/ADC6)
Changed lines of the file:
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@@
+	(wire
+		(pts
+			(xy 102.87 170.18) (xy 113.03 170.18)
+		)
+		(stroke
+			(width 0)
+			(type default)
+		)
+	)
 	(wire
 		(pts
@@
 		)
 	)
+	(label "EXPANDER_INT"
+		(at 102.87 170.18 180)
+		(effects
+			(font
+				(size 1.27 1.27)
+			)
+			(justify right bottom)
+		)
+	)

Commit message: 12th
Parts:
- added R49, R50: 33, Resistor_SMD:R_0402_1005Metric, symbol Device:R
Connections:
- net BLE_UART_RXD: now also R50.2; no longer U2.33 (UART_RXD)
- net BLE_UART_TXD: now also R49.2; no longer U2.32 (UART_TXD)
- new net: R49.1, U2.32 (UART_TXD)
- new net: R50.1, U2.33 (UART_RXD)
Changed lines of the file:
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@@
 	(wire
 		(pts
+			(xy 373.38 210.82) (xy 374.65 210.82)
+		)
+		(stroke
+			(width 0)
+			(type default)
+		)
+	)
+	(wire
+		(pts
 			(xy 284.48 67.31) (xy 289.56 67.31)
 		)
@@
 	(wire
 		(pts
-			(xy 356.87 210.82) (xy 367.03 210.82)
+			(xy 356.87 210.82) (xy 365.76 210.82)
 		)
 		(stroke
@@
 	(wire
 		(pts
-			(xy 356.87 213.36) (xy 367.03 213.36)
+			(xy 356.87 213.36) (xy 375.285 213.36)
 		)
 		(stroke
@@
 	(wire
 		(pts
+			(xy 358.14 208.28) (xy 356.87 208.28)
+		)
+		(stroke
+			(width 0)
+			(type default)
+		)
+	)
+	(wire
+		(pts
 			(xy 39.37 194.31) (xy 43.18 194.31)
 		)
@@
 	(wire
 		(pts
-			(xy 367.03 208.28) (xy 356.87 208.28)
+			(xy 374.65 208.28) (xy 365.76 208.28)
 		)
 		(stroke
@@
 	)
 	(label "BLE_UART_TXD"
-		(at 367.03 208.28 0)
+		(at 374.65 208.28 0)
 		(effects
 			(font
@@
 	)
 	(label "BLE_UART_CTS"
-		(at 367.03 213.36 0)
+		(at 375.285 213.36 0)
 		(effects
 			(font
@@
 	)
 	(label "BLE_UART_RXD"
-		(at 367.03 210.82 0)
+		(at 374.65 210.82 0)
 		(effects
 			(font
@@
 	)
 	(symbol
+		(lib_id "Device:R")
+		(at 361.95 208.28 90)
+		(unit 1)
+		(body_style 1)
+		(exclude_from_sim no)
+		(in_bom yes)
+		(on_board yes)
+		(in_pos_files yes)
+		(dnp no)
+		(property "Reference" "R49"
+			(at 361.95 202.565 90)
+			(show_name no)
+			(do_not_autoplace no)
+			(effects
+				(font
+					(size 1.27 1.27)
+				)
+			)
+		)
+		(property "Value" "33"
+			(at 361.95 205.105 90)
+			(show_name no)
+			(do_not_autoplace no)
+			(effects
+				(font
+					(size 1.27 1.27)
+				)
+			)
+		)
+		(property "Footprint" "Resistor_SMD:R_0402_1005Metric"
+			(at 361.95 210.058 90)
+			(hide yes)
+			(show_name no)
+			(do_not_autoplace no)
+			(effects
+				(font
+					(size 1.27 1.27)
+				)
+			)
+		)
+		(property "Datasheet" ""
+			(at 361.95 208.28 0)
+			(hide yes)
+			(show_name no)
+			(do_not_autoplace no)
+			(effects
+				(font
+					(size 1.27 1.27)
+				)
+			)
+		)
+		(property "Description" "Resistor"
+			(at 361.95 208.28 0)
+			(hide yes)
+			(show_name no)
+			(do_not_autoplace no)
+			(effects
+				(font
+					(size 1.27 1.27)
+				)
+			)
+		)
+		(property "LCSC Part" "C25105"
+			(at 361.95 208.28 90)
+			(hide yes)
+			(show_name no)
+			(do_not_autoplace no)
+			(effects
+				(font
+					(size 1.27 1.27)
+				)
+			)
+		)
+		(pin "2"
+		)
+		(pin "1"
+		)
+		(instances
+			(project "mp3player"
+				(path "/730d0887-0a09-4397-bcb4-2959d410b5ba/e503cbcc-34c8-46b6-97a8-cd1a740433c3"
+					(reference "R49")
+					(unit 1)
+				)
+			)
+		)
+	)
+	(symbol
 		(lib_id "power:GND")
 		(at 351.79 184.15 90)
@@
 					(unit 1)
 				)
+			)
+		)
+	)
+	(symbol
+		(lib_id "Device:R")
+		(at 369.57 210.82 90)
+		(unit 1)
+		(body_style 1)
+		(exclude_from_sim no)
+		(in_bom yes)
+		(on_board yes)
+		(in_pos_files yes)
+		(dnp no)
+		(property "Reference" "R50"
+			(at 369.57 205.105 90)
+			(show_name no)
+			(do_not_autoplace no)
+			(effects
+				(font
+					(size 1.27 1.27)
+				)
+			)
+		)
+		(property "Value" "33"
+			(at 369.57 207.645 90)
+			(show_name no)
+			(do_not_autoplace no)
+			(effects
+				(font
+					(size 1.27 1.27)
+				)
+			)
+		)
+		(property "Footprint" "Resistor_SMD:R_0402_1005Metric"
+			(at 369.57 212.598 90)
+			(hide yes)
+			(show_name no)
+			(do_not_autoplace no)
+			(effects
+				(font
+					(size 1.27 1.27)
+				)
+			)
+		)
+		(property "Datasheet" ""
+			(at 369.57 210.82 0)
+			(hide yes)
+			(show_name no)
+			(do_not_autoplace no)
+			(effects
+				(font
+					(size 1.27 1.27)
+				)
+			)
+		)
+		(property "Description" "Resistor"
+			(at 369.57 210.82 0)
+			(hide yes)
+			(show_name no)
+			(do_not_autoplace no)
+			(effects
+				(font
+					(size 1.27 1.27)
+				)
+			)
+		)
+		(property "LCSC Part" "C25105"
+			(at 369.57 210.82 90)
+			(hide yes)
+			(show_name no)
+			(do_not_autoplace no)
+			(effects
+				(font
+					(size 1.27 1.27)
+				)
+			)
+		)
+		(pin "2"
+		)
+		(pin "1"
+		)
+		(instances
+			(project "mp3player"
+				(path "/730d0887-0a09-4397-bcb4-2959d410b5ba/e503cbcc-34c8-46b6-97a8-cd1a740433c3"
+					(reference "R50")
+					(unit 1)
+				)

Commit message: pcb updates + journaling
Parts:
- added D4: LED, LED_SMD:LED_0603_1608Metric, symbol Device:LED
- added R51: 330, Resistor_SMD:R_0402_1005Metric, symbol Device:R
- J3: LCSC Part (none) -> //; now left out of the parts list
Connections:
- net GND: now also D4.1 (K)
- net at U6.58 (GPIO47/ADC7): now also R51.2
- new net: D4.2 (A), R51.1

Commit message: firmware/journal update
Connections:
- net DB10: now also U6.37 (GPIO29); no longer U6.38 (GPIO30)
- net DB11: now also U6.38 (GPIO30); no longer U6.39 (GPIO31)
- net DB12: now also U6.39 (GPIO31); no longer U6.40 (GPIO32)
- net DB13: now also U6.40 (GPIO32); no longer U6.42 (GPIO33)
- net DB14: now also U6.42 (GPIO33); no longer U6.43 (GPIO34)
- net DB15: now also U6.43 (GPIO34); no longer U6.44 (GPIO35)
- net DB16: now also U6.44 (GPIO35); no longer U6.45 (GPIO36)
- net DB17: now also U6.45 (GPIO36); no longer U6.46 (GPIO37)
- net DB5: no longer U6.26 (GPIO25)
- net DB6: now also U6.26 (GPIO25); no longer U6.27 (GPIO26)
- net DB7: now also U6.27 (GPIO26); no longer U6.28 (GPIO27)
- net DB8: now also U6.28 (GPIO27); no longer U6.36 (GPIO28)
- net DB9: now also U6.36 (GPIO28); no longer U6.37 (GPIO29)
- net GPIO26 renamed SD_CLK
- net SD_CLK: now also U6.49 (GPIO40/ADC0); no longer U6.56 (GPIO45/ADC5)
- net GPIO27 renamed SD_CMD
- net SD_CMD: now also U6.52 (GPIO41/ADC1); no longer U6.55 (GPIO44/ADC4)
- net GPIO28 renamed SD_DAT0
- net SD_DAT0: now also U6.53 (GPIO42/ADC2); no longer U6.54 (GPIO43/ADC3)
- net GPIO29 renamed SD_DAT1
- net SD_DAT1: now also U6.54 (GPIO43/ADC3); no longer U6.53 (GPIO42/ADC2)
- net GPIO30 renamed SD_DAT2
- net SD_DAT2: now also U6.55 (GPIO44/ADC4); no longer U6.52 (GPIO41/ADC1)
- net GPIO31 renamed SD_DAT3
- net SD_DAT3: now also U6.56 (GPIO45/ADC5); no longer U6.49 (GPIO40/ADC0)

Commit message: cad added + journal/bom update
Parts:
- C2: LCSC Part C23733 -> C368809
- C24, C25, C55: LCSC Part C52923 -> C307427
- R1, R32, R33, R38, R48, R49, R50: LCSC Part C25105 -> C2906931
- R10, R11, R12, R29, R35, R47, R5, R7, R8, R9: LCSC Part C25744 -> C2906861
- R34: value 5 -> 6.8; LCSC Part C25197 -> C2907056
- R36, R37: LCSC Part C25900 -> C2906941
- R4, R6: LCSC Part C11702 -> C852624
- R51: LCSC Part C25104 -> C71626
Other:
- note added: "6.8ohm would be optimal but no jlcpcb basic part so expensive"
Changed lines of the file:
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@@
 		)
 	)
+	(text "6.8ohm would be optimal\nbut no jlcpcb basic part so expensive"
+		(exclude_from_sim no)
+		(at 476.885 65.405 0)
+		(effects
+			(font
+				(size 1.27 1.27)
+			)
+		)
+	)
 	(text "1\n"
 		(exclude_from_sim no)
@@
 			)
 		)
-		(property "LCSC Part" "C25744"
+		(property "LCSC Part" "C2906861"
 			(at 434.34 198.12 90)
 			(hide yes)
@@
 			)
 		)
-		(property "LCSC Part" "C25105"
+		(property "LCSC Part" "C2906931"
 			(at 361.95 208.28 90)
 			(hide yes)
@@
 			)
 		)
-		(property "Value" "5"
+		(property "Value" "6.8"
 			(at 457.2 60.9599 0)
 			(show_name no)
@@
 			)
 		)
-		(property "LCSC Part" "C25197"
+		(property "LCSC Part" "C2907056"
 			(at 454.66 59.69 0)
 			(hide yes)
@@
 			)
 		)
-		(property "LCSC Part" "C25744"
+		(property "LCSC Part" "C2906861"
 			(at 333.375 55.88 0)
 			(hide yes)
@@
 			)
 		)
-		(property "LCSC Part" "C52923"
+		(property "LCSC Part" "C307427"
 			(at 469.9 48.26 0)
 			(hide yes)
@@
 			)
 		)
-		(property "LCSC Part" "C25105"
+		(property "LCSC Part" "C2906931"
 			(at 170.815 88.9 90)
 			(hide yes)
@@
 			)
 		)
-		(property "LCSC Part" "C25900"
+		(property "LCSC Part" "C2906941"
 			(at 179.07 180.34 0)
 			(hide yes)
@@
 			)
 		)
-		(property "LCSC Part" "C11702"
+		(property "LCSC Part" "C852624"
 			(at 39.37 171.45 0)
 			(hide yes)
@@
 			)
 		)
-		(property "LCSC Part" "C25744"
+		(property "LCSC Part" "C2906861"
 			(at 421.64 226.06 90)
 			(hide yes)
@@
 			)
 		)
-		(property "LCSC Part" "C11702"
+		(property "LCSC Part" "C852624"
 			(at 193.04 267.97 90)
 			(hide yes)
@@
 			)
 		)
-		(property "LCSC Part" "C25105"
+		(property "LCSC Part" "C2906931"
 			(at 170.815 96.52 90)
 			(hide yes)
@@
 			)
 		)
-		(property "LCSC Part" "C52923"
+		(property "LCSC Part" "C307427"
 			(at 331.47 180.34 90)
 			(hide yes)
@@
 			)
 		)
-		(property "LCSC Part" "C25105"
+		(property "LCSC Part" "C2906931"
 			(at 170.815 91.44 90)
 			(hide yes)
@@
 			)
 		)
-		(property "LCSC Part" "C25105"
+		(property "LCSC Part" "C2906931"
 			(at 369.57 210.82 90)
 			(hide yes)
@@
 			)
 		)
-		(property "LCSC Part" "C25104"
+		(property "LCSC Part" "C71626"
 			(at 97.155 177.8 0)
 			(hide yes)
@@
 			)
 		)
-		(property "LCSC Part" "C25105"
+		(property "LCSC Part" "C2906931"
 			(at 170.815 93.98 90)
 			(hide yes)
@@
 			)
 		)
-		(property "LCSC Part" "C52923"
+		(property "LCSC Part" "C307427"
 			(at 346.71 184.15 90)
 			(hide yes)
@@
 			)
 		)
-		(property "LCSC Part" "C25744"
+		(property "LCSC Part" "C2906861"
 			(at 369.57 229.87 0)
 			(hide yes)
@@
 			)
 		)
-		(property "LCSC Part" "C25744"
+		(property "LCSC Part" "C2906861"
 			(at 414.02 200.66 90)
 			(hide yes)
@@
 			)
 		)
-		(property "LCSC Part" "C25744"
+		(property "LCSC Part" "C2906861"
 			(at 481.965 213.995 0)
 			(hide yes)
@@
 			)
 		)
-		(property "LCSC Part" "C25900"
+		(property "LCSC Part" "C2906941"
 			(at 170.18 177.8 0)
 			(hide yes)
@@
 			)
 		)
-		(property "LCSC Part" "C25744"
+		(property "LCSC Part" "C2906861"
 			(at 105.41 236.22 0)
 			(hide yes)
@@
 			)
 		)
-		(property "LCSC Part" "C25744"
+		(property "LCSC Part" "C2906861"
 			(at 284.48 73.66 0)
 			(hide yes)
@@
 			)
 		)
-		(property "LCSC Part" "C25744"
+		(property "LCSC Part" "C2906861"
 			(at 420.37 195.58 90)
 			(hide yes)
@@
 			)
 		)
-		(property "LCSC Part" "C23733"
+		(property "LCSC Part" "C368809"
 			(at 36.83 260.35 0)
 			(hide yes)
@@
 			)
 		)
-		(property "LCSC Part" "C25744"
+		(property "LCSC Part" "C2906861"
 			(at 410.21 210.82 90)
 			(hide yes)
@@
 			)
 		)
-		(property "LCSC Part" "C25105"
+		(property "LCSC Part" "C2906931"
 			(at 38.1 240.03 90)
 			(hide yes)
