File: src/kicad/mp3player.kicad_pcb (KiCad board)
At the start: 2 copper layers, 2 x 5.3 mm, 134 parts, among them J1 SD_Card_Receptacle, J2 USB_C_Receptacle_USB2.0_16P, J5 Conn_01x02, J6 Conn_01x42, J7 AudioJack3_Ground_SwitchTR, Q2 BSS138, Q3 BSS138, Q4 BSS138, SW1 EVQPUL02K, SW10 EVQPUL02K, SW11 TS-1088-AR02016, SW3 SW_Push, SW4 SW_Push, SW5 SW_Push, SW7 EVQPUL02K, SW8 SW_Push, SW9 SW_Push, U1 ABM8-272-T3_C20625731, U10 LP5907MFX-3.3, U11 TPS61165DRV, U12 TCA9555RTWR, U3 W25Q128JVE, U4 APS6404L-SQRx-ZR, U5 PCM5102A, U6 RP2350B, U7 TPS63070RNMR, U8 BQ24075RGT, U9 MAX17048G_T10

Commit message: routing + may 30th update + things
Parts:
- C26, C28, C29, C30, C39, C40, C42, C43, C44, C45, C46, C48, C49, C50, C51, C52, C56, C57, J1, J2, J5, J6, J7, Q2, Q4, R13, R14, R15, R16, R17, R22, R23, R24, R25, R30, R31, R39, SW1, SW10, SW7, U10, U5, U8: moved to B.Cu
- C41: value 1uf -> 4.7uf; footprint Capacitor_SMD:C_0402_1005Metric -> Capacitor_SMD:C_0603_1608Metric; moved to B.Cu
- moved U6 160.8 mm to (123.9, 189.2), turned to 180 degrees
- moved C27 127.2 mm to (163.3, 123.0)
- moved C32 127.2 mm to (163.3, 126.9)
- moved C33 127.2 mm to (139.1, 130.8)
- moved C34 127.2 mm to (143.1, 123.3)
- moved C35 127.2 mm to (143.1, 125.8)
- moved C37 127.2 mm to (143.1, 130.8)
- moved D1 127.2 mm to (159.8, 115.4)
- moved L1 127.2 mm to (178.8, 110.8)
- moved L2 127.2 mm to (161.4, 140.7)
- moved R34 127.2 mm to (164.7, 117.5)
- moved R40 127.2 mm to (194.8, 75.5)
- moved R41 127.2 mm to (194.8, 77.5)
- moved R43 127.2 mm to (194.8, 81.5)
- moved R44 127.2 mm to (194.8, 83.4)
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Connections:
- R40 pad 2: /processing/DPAD.DOWN -> /processing/VOLUME.DOWN
- R41 pad 2: /processing/DPAD.UP -> /processing/VOLUME.UP
- R42 pad 1: /processing/VOLUME.DOWN -> /processing/DPAD.DOWN
- R43 pad 1: /processing/VOLUME.UP -> /processing/DPAD.UP
- R44 pad 1: /ui/DPAD.LEFT -> /processing/DPAD.LEFT
- R45 pad 1: /ui/DPAD.RIGHT -> /processing/DPAD.RIGHT
- R46 pad 1: /ui/DPAD.CENTER -> /processing/DPAD.CENTER
- SW10 pad 1: GND -> /processing/VOLUME.DOWN
- SW10 pad 2: /processing/DPAD.DOWN -> GND
- SW3 pad 1: /ui/DPAD.CENTER -> /processing/DPAD.CENTER
- SW4 pad 2: /processing/VOLUME.UP -> /processing/DPAD.UP
- SW5 pad 1: /processing/VOLUME.DOWN -> /processing/DPAD.DOWN
- SW7 pad 2: /processing/DPAD.UP -> /processing/VOLUME.UP
- SW8 pad 1: /ui/DPAD.RIGHT -> /processing/DPAD.RIGHT
- SW9 pad 1: /ui/DPAD.LEFT -> /processing/DPAD.LEFT
Routing:
- net GND: track 0.00 -> 84.5 mm, vias 0 -> 34
- net /audio/SW_T: track 0.00 -> 39.2 mm, vias 0 -> 2
- net /power/USB_VBUS: track 0.00 -> 31.3 mm, vias 0 -> 2
- net /audio/+3V3_ANALOG: track 0.00 -> 26.1 mm, vias 0 -> 2
- net +3V3: track 0.00 -> 23.4 mm, vias 0 -> 6
- net /power/LIPO_+: track 0.00 -> 17.5 mm
- net Net-(Q2-D): track 0.00 -> 13.1 mm, vias 0 -> 2
- net /audio/LEFT_AUDIO: track 0.00 -> 12.3 mm
- net /power/B_EN2: track 0.00 -> 9.77 mm
- net Net-(U5-XSMT): track 0.00 -> 6.95 mm
- net Net-(U5-OUTL): track 0.00 -> 5.23 mm
- net Net-(U5-OUTR): track 0.00 -> 4.99 mm
- net Net-(U5-LDOO): track 0.00 -> 4.96 mm
- net Net-(U5-CAPM): track 0.00 -> 4.69 mm
- net /audio/RIGHT_AUDIO: track 0.00 -> 4.11 mm
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- added copper zone on In2.Cu, net +3V3
- added copper zone on In1.Cu, net GND
Other:
- board size 2 x 5.3 mm -> 52 x 115.8 mm
- copper layers 2 -> 4

Commit message: jun 1st what already noo
Parts:
- added C47: 100nf, Capacitor_SMD:C_0402_1005Metric, B.Cu at (63.1, 107.9)
- added J4: Conn_01x03, Connector_PinHeader_2.54mm:PinHeader_1x03_P2.54mm_Vertical, F.Cu at (98.8, 47.8)
- added U2: FSC-BT1114QI, feasycom:FSC-BT1114QI, B.Cu at (39.3, 85.7)
- C1, C10, C11, C12, C13, C14, C15, C2, C20, C21, C27, C3, C31, C32, C33, C34, C35, C36, C37, C38, C4, C5, C53, C54, C55, C6, C7, C8, C9, D1, D2, D3, L1, L2, L3, Q3, R1, R18, R2, R20, R21, R26, R27, R28, R3, R34, R6, U1, U11, U12, U3, U4, U6, U7, U9: moved to B.Cu
- R19: value 10k -> 100k; moved to B.Cu
- moved U11 144.8 mm to (39.9, 78.0), turned to -90 degrees
- moved C54 137.4 mm to (41.0, 75.4), turned to 90 degrees
- moved C53 133.4 mm to (35.0, 83.6)
- moved R34 133.3 mm to (38.4, 74.8), turned to 90 degrees
- moved C55 133.1 mm to (45.5, 74.4)
- moved Q3 130.3 mm to (64.9, 51.0)
- moved U4 127.4 mm to (52.1, 109.2), turned to -80 degrees
- moved D3 125.9 mm to (64.6, 54.8)
- moved L2 124.3 mm to (67.5, 59.2)
- moved R28 122.2 mm to (67.3, 52.6), turned to 180 degrees
- moved D1 122.1 mm to (44.1, 76.2), turned to 180 degrees
- moved D2 119.9 mm to (69.8, 54.8), turned to 180 degrees
- moved R27 119.2 mm to (69.6, 52.6), turned to 180 degrees
- moved L3 118.9 mm to (39.8, 82.0)
- moved R26 118.6 mm to (69.6, 51.4)
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Connections:
- U7 pad 15: +3V3 -> GND
Routing:
- net /power/USB_D-: track 2.61 -> 85.6 mm, vias 0 -> 2
- net /power/USB_D+: track 2.54 -> 85.3 mm, vias 0 -> 2
- net /power/LIPO_+: track 17.5 -> 85.4 mm, vias 0 -> 3
- net GND: track 84.5 -> 145.2 mm, vias 34 -> 83
- net +3V3: track 23.4 -> 56.9 mm, vias 6 -> 13
- net /power/B_EN2: track 9.77 -> 31.9 mm
- net /processing/LED_K: track 0.00 -> 22.0 mm
- net /processing/QSPI_SD3: track 0.00 -> 17.9 mm
- net /processing/QSPI_SD1: track 0.00 -> 17.7 mm
- net /processing/QSPI_SD2: track 0.00 -> 17.7 mm
- net /audio/SW_T: track 39.2 -> 56.1 mm, vias 2 -> 1
- net Net-(D2-A): track 0.00 -> 16.7 mm
- net /processing/QSPI_CLK: track 0.00 -> 15.7 mm
- net /processing/QSPI_SD0: track 0.00 -> 13.6 mm
- net /processing/QSPI_SS: track 0.00 -> 12.7 mm
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- added copper zone on B.Cu, net +1V1
- added copper zone on B.Cu, net +3V3
- added copper zone on B.Cu, net /processing/VREG_LX
- added copper zone on B.Cu, net GND

Commit message: first of june wo&
Parts:
- removed C17, C18: 100nf, Capacitor_SMD:C_0402_1005Metric
- C16, C19, C22, C23, C24, C25, J4, R10, R11, R12, R29, R35, R36, R37, R4, R47, R5, R7, R8, R9, SW11: moved to B.Cu
- moved SW3 139.2 mm to (57.2, 139.8)
- moved SW5 137.9 mm to (57.2, 152.9)
- moved C24 135.1 mm to (43.4, 88.7), turned to 180 degrees
- moved C25 134.6 mm to (45.6, 105.0), turned to 180 degrees
- moved C22 134.5 mm to (63.1, 145.3), turned to -90 degrees
- moved C23 129.8 mm to (50.4, 100.2), turned to 90 degrees
- moved SW9 128.5 mm to (44.0, 139.8)
- moved C19 128.2 mm to (50.0, 110.6), turned to 45 degrees
- moved C16 125.9 mm to (54.3, 112.5), turned to 180 degrees
- moved SW4 124.2 mm to (57.2, 126.5)
- moved R12 123.7 mm to (49.0, 103.5), turned to -135 degrees
- moved R11 119.6 mm to (62.2, 155.8), turned to 180 degrees
- moved R5 119.4 mm to (50.2, 107.8), turned to 90 degrees
- moved R10 117.7 mm to (63.4, 151.7), turned to -135 degrees
- moved R4 117.5 mm to (52.1, 104.1), turned to 45 degrees
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Connections:
- U6 pad 9: unconnected-(U6-GPIO11-Pad9) -> /processing/DISPLAY_RESET
Routing:
- net /audio/ANALOG_LDO_EN: track 1.62 -> 97.3 mm, vias 0 -> 2
- net /audio/JACK_DETECTION: track 1.97 -> 88.9 mm, vias 0 -> 2
- net /power/POWER_BTN_SENSE: track 2.35 -> 82.7 mm, vias 0 -> 2
- net /processing/GPIO29: track 0.00 -> 73.5 mm
- net /processing/GPIO28: track 0.00 -> 70.2 mm
- net /processing/GPIO26: track 0.00 -> 58.8 mm
- net /processing/GPIO27: track 0.00 -> 53.8 mm
- net GND: track 145.2 -> 198.2 mm, vias 83 -> 115
- net /processing/CARD_DETECT: track 0.00 -> 52.7 mm, vias 0 -> 2
- net /processing/GPIO31: track 0.00 -> 48.8 mm
- net /processing/GPIO30: track 0.00 -> 45.5 mm
- net /processing/DB17: track 0.00 -> 43.5 mm
- net /processing/DB16: track 0.00 -> 42.9 mm
- net /processing/DB15: track 0.00 -> 42.3 mm
- net /processing/DB14: track 0.00 -> 41.7 mm
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
Commit message: new dayy
Parts:
- removed J4: Conn_01x03, Connector_PinHeader_2.54mm:PinHeader_1x03_P2.54mm_Vertical
- added J3: Conn_01x05, misc:test_pads, B.Cu at (42.4, 118.2)
- added R32: 33, Resistor_SMD:R_0402_1005Metric, B.Cu at (58.1, 100.0)
- added R33: 33, Resistor_SMD:R_0402_1005Metric, B.Cu at (58.8, 99.3)
- added R38: 33, Resistor_SMD:R_0402_1005Metric, B.Cu at (59.5, 98.6)
- added R48: 33, Resistor_SMD:R_0402_1005Metric, B.Cu at (60.2, 97.9)
- R40, R41, R42, R43, R44, R45, R46: moved to B.Cu
- moved R41 115.1 mm to (33.3, 70.1), turned to 180 degrees
- moved R40 108.9 mm to (33.5, 81.0), turned to 45 degrees
- moved R42 72.5 mm to (64.4, 155.4), turned to -90 degrees
- moved R46 71.0 mm to (61.7, 132.4)
- moved R43 70.5 mm to (62.1, 128.2), turned to 90 degrees
- moved R44 67.4 mm to (66.4, 147.4), turned to -90 degrees
- moved R45 59.1 mm to (73.4, 136.5), turned to 180 degrees
- moved R31 5.10 mm to (56.6, 49.5), turned to 90 degrees
- moved C53 4.08 mm to (38.8, 85.2), turned to 180 degrees
- moved C26 2.75 mm to (56.9, 53.9)
- moved Q4 1.59 mm to (59.3, 48.9)
- moved C34 0.92 mm to (61.0, 61.0), turned to 180 degrees
- moved C36 0.91 mm to (61.0, 64.1), turned to 180 degrees
- moved C35 0.34 mm to (59.9, 62.5)
Connections:
- U6 pad 3: /audio/I2S.DIN -> Net-(U6-GPIO6)
- U6 pad 35: unconnected-(U6-RUN-Pad35) -> /processing/RUN
- U6 pad 4: /audio/I2S.BCK -> Net-(U6-GPIO7)
- U6 pad 6: /audio/I2S.LRCK -> Net-(U6-GPIO8)
- U6 pad 7: /audio/I2S.SCK -> Net-(U6-GPIO9)
Routing:
- net /audio/I2S.LRCK: track 0.00 -> 109.8 mm, vias 0 -> 2
- net /processing/VOLUME.UP: track 0.00 -> 107.2 mm, vias 0 -> 2
- net /audio/I2S.SCK: track 0.00 -> 95.6 mm, vias 0 -> 2
- net /processing/VOLUME.DOWN: track 0.00 -> 93.4 mm, vias 0 -> 2
- net /audio/I2S.BCK: track 0.00 -> 90.1 mm, vias 0 -> 2
- net /audio/I2S.DIN: track 0.00 -> 89.8 mm, vias 0 -> 2
- net /processing/RUN: track 0.00 -> 88.4 mm, vias 0 -> 2
- net /processing/RP_SWDIO: track 0.00 -> 86.8 mm, vias 0 -> 2
- net /processing/RP_SWCLK: track 0.00 -> 81.2 mm, vias 0 -> 2
- net /processing/DPAD.LEFT: track 0.00 -> 74.5 mm, vias 0 -> 1
- net /power/POWER_GPIO: track 0.00 -> 71.1 mm, vias 0 -> 2
- net /processing/DPAD.DOWN: track 0.00 -> 63.9 mm, vias 0 -> 1
- net /power/B_EN2: track 31.9 -> 88.3 mm, vias 0 -> 1
- net /power/CHG_PIN: track 3.43 -> 56.9 mm, vias 1 -> 2
- net /processing/DPAD.CENTER: track 0.00 -> 50.5 mm, vias 0 -> 3
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Other:
- outline, holes or cut-outs redrawn

Commit message: new day!
Connections:
- U6 pad 57: unconnected-(U6-GPIO46/ADC6-Pad57) -> /processing/EXPANDER_INT
Routing:
- net GND: track 206.7 -> 208.7 mm, vias 135 -> 132
- net /processing/CARD_DETECT: track 52.2 -> 54.0 mm
- net /processing/EXPANDER_INT: track 13.6 -> 12.4 mm
- net /processing/SPI.SDA: track 29.3 -> 30.4 mm
- net /power/B_EN2: track 88.3 -> 87.3 mm, vias 1 -> 0
- net /power/POWER_BTN_SENSE: track 71.2 -> 70.3 mm, vias 5 -> 4
- net +3V3: track 100.9 -> 101.7 mm, vias 47 -> 46
- net /processing/GPIO30: track 45.5 -> 46.3 mm
- net /processing/GPIO26: track 58.8 -> 59.4 mm
- net /processing/GPIO27: track 53.8 -> 54.4 mm
- net /processing/DISPLAY_RESET: track 30.1 -> 29.6 mm
- net /processing/GPIO29: track 73.5 -> 74.0 mm
Other:
- outline, holes or cut-outs redrawn

Commit message: 12th
Parts:
- added R49: 33, Resistor_SMD:R_0402_1005Metric, B.Cu at (39.7, 105.4)
- added R50: 33, Resistor_SMD:R_0402_1005Metric, B.Cu at (55.3, 101.6)
- moved SW11 10.5 mm to (34.0, 122.9)
- moved R40 3.37 mm to (34.2, 77.7), turned to 180 degrees
- moved SW10 2.79 mm to (33.3, 73.4)
- moved SW7 2.45 mm to (33.2, 63.1)
- moved R41 2.45 mm to (33.4, 67.6)
- moved J3 1.99 mm to (44.4, 118.3)
- moved C23 1.00 mm to (50.5, 99.2)
- moved U2 0.13 mm to (39.4, 85.1)
Connections:
- U2 pad 32: /processing/BLE_UART_TXD -> Net-(U2-UART_TXD)
- U2 pad 33: /processing/BLE_UART_RXD -> Net-(U2-UART_RXD)
Routing:
- net /processing/RP_SWDIO: track 86.9 -> 59.9 mm
- net /processing/RUN: track 88.7 -> 62.0 mm
- net /processing/BLE_UART_RXD: track 31.7 -> 6.10 mm
- net /processing/RP_SWCLK: track 81.2 -> 55.6 mm
- net Net-(U2-UART_RXD): track 0.00 -> 25.4 mm
- net /audio/I2S.LRCK: track 110.1 -> 92.3 mm
- net Net-(R4-Pad1): track 21.1 -> 31.6 mm
- net /processing/VOLUME.DOWN: track 93.4 -> 103.5 mm, vias 2 -> 4
- net /audio/I2S.SCK: track 95.6 -> 100.9 mm
- net /processing/EXPANDER_INT: track 12.4 -> 16.3 mm
- net GND: track 208.7 -> 212.6 mm, vias 132 -> 124
- net /processing/VOLUME.UP: track 107.2 -> 103.8 mm, vias 2 -> 4
- net /audio/I2S.DIN: track 89.8 -> 86.9 mm
- net /processing/BLE_UART_TXD: track 32.1 -> 29.6 mm
- net /audio/I2S.BCK: track 90.1 -> 87.7 mm
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- added copper zone on In1.Cu, net +3V3
- added copper zone on In2.Cu, net GND
- removed copper zone on In2.Cu, net +3V3
- removed copper zone on In1.Cu, net GND
Other:
- outline, holes or cut-outs redrawn

Commit message: pcb updates + journaling
Parts:
- added D4: LED, LED_SMD:LED_0603_1608Metric, B.Cu at (82.2, 52.7)
- added R51: 330, Resistor_SMD:R_0402_1005Metric, B.Cu at (81.7, 56.0)
- added REF**: MountingHole_2.2mm_M2, MountingHole:MountingHole_2.2mm_M2, F.Cu at (34.0, 116.5)
- added REF**: MountingHole_2.2mm_M2, MountingHole:MountingHole_2.2mm_M2, F.Cu at (38.1, 63.8)
- added REF**: MountingHole_2.2mm_M2, MountingHole:MountingHole_2.2mm_M2, F.Cu at (70.2, 71.9)
- moved R8 1.15 mm to (64.9, 137.5)
- moved R14 1.12 mm to (76.7, 54.6)
- moved R46 1.10 mm to (61.6, 131.3)
- moved Q3 1.07 mm to (63.8, 51.0)
- moved J2 1.05 mm to (75.2, 50.1)
- moved SW1 1.03 mm to (65.0, 46.6)
- moved R11 0.97 mm to (62.5, 154.9)
- moved R28 0.94 mm to (66.4, 52.3), turned to -90 degrees
- moved R27 0.85 mm to (68.8, 52.6)
- moved R26 0.83 mm to (68.8, 51.5)
- moved R9 0.77 mm to (63.0, 135.7)
- moved R13 0.75 mm to (73.8, 54.6)
- moved J1 0.73 mm to (50.1, 143.6)
- moved C22 0.60 mm to (63.1, 144.7)
- moved R7 0.55 mm to (63.0, 140.0)
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Connections:
- U6 pad 58: unconnected-(U6-GPIO47/ADC7-Pad58) -> Net-(U6-GPIO47/ADC7)
Routing:
- net Net-(U6-GPIO47/ADC7): track 0.00 -> 92.8 mm, vias 0 -> 2
- net GND: track 212.6 -> 220.8 mm, vias 124 -> 127
- net Net-(D4-A): track 0.00 -> 4.79 mm
- net /power/USB_D+: track 89.4 -> 92.1 mm
- net /power/USB_VBUS: track 33.0 -> 35.1 mm
- net Net-(D2-A): track 16.7 -> 18.7 mm
- net /processing/GPIO30: track 46.3 -> 44.2 mm
- net /processing/GPIO31: track 49.3 -> 47.5 mm
- net /power/LIPO_+: track 58.6 -> 60.2 mm
- net /processing/GPIO27: track 54.4 -> 52.9 mm
- net /processing/GPIO29: track 74.0 -> 72.7 mm
- net /power/B_EN2: track 87.3 -> 86.0 mm
- net /processing/DPAD.CENTER: track 50.5 -> 51.3 mm
- net /processing/GPIO26: track 59.4 -> 58.7 mm
Other:
- board size 52 x 115.8 mm -> 52 x 115.7 mm

Commit message: journal & files update
Parts:
- removed the REF** at (34.0, 116.5)
- moved R45 7.40 mm to (75.6, 129.4), turned to 0 degrees
- moved SW3 3.21 mm to (57.2, 136.5)
- moved SW5 3.21 mm to (57.2, 149.7)
- moved SW8 3.21 mm to (70.4, 136.6)
- moved SW9 3.21 mm to (44.0, 136.5)
- moved SW4 3.21 mm to (57.2, 123.3)
- moved R34 2.25 mm to (40.6, 74.8)
- moved SW1 2.22 mm to (65.2, 48.8)
- moved SW7 2.04 mm to (35.3, 63.2)
- moved SW10 2.03 mm to (35.3, 73.5)
- moved REF** 1.91 mm to (39.8, 62.9)
- moved Q3 1.64 mm to (63.6, 52.6), turned to 180 degrees
- moved C54 1.53 mm to (42.5, 75.2)
- moved U11 1.25 mm to (41.1, 77.9)
- moved C55 0.92 mm to (46.4, 74.2), turned to -90 degrees
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Routing:
- net GND: track 220.8 -> 231.1 mm, vias 127 -> 123
- net /processing/DPAD.CENTER: track 51.3 -> 46.9 mm
- net /processing/DPAD.RIGHT: track 38.5 -> 34.5 mm
- net Net-(D2-A): track 18.7 -> 15.4 mm
- net /processing/LED_K: track 22.0 -> 18.8 mm
- net Net-(D1-A): track 9.71 -> 6.59 mm
- net /power/B_EN2: track 86.0 -> 83.5 mm
- net Net-(D3-K): track 2.90 -> 4.64 mm
- net /processing/LED_A: track 4.73 -> 6.40 mm
- net /processing/CARD_DETECT: track 53.6 -> 55.2 mm
- net /power/LIPO_+: track 60.2 -> 58.9 mm
- net /audio/JACK_DETECTION: track 79.9 -> 81.0 mm
- net /power/POWER_BTN_SENSE: track 70.4 -> 71.2 mm, vias 4 -> 5
- net /processing/DPAD.DOWN: track 63.9 -> 64.7 mm
- net /processing/DPAD.UP: track 42.5 -> 43.2 mm
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Other:
- outline, holes or cut-outs redrawn
