File: src/kicad/mp3player.kicad_pcb (KiCad board)
At the start: 4 copper layers, 52 x 115.7 mm, 145 parts, among them J1 SD_Card_Receptacle, J2 USB_C_Receptacle_USB2.0_16P, J3 Conn_01x05, J5 Conn_01x02, J6 Conn_01x42, J7 AudioJack3_Ground_SwitchTR, Q2 BSS138, Q3 BSS138, Q4 BSS138, SW1 EVQPUL02K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

Commit message: june 18th update
Parts:
- added REF**: MountingHole_2.2mm_M2, MountingHole:MountingHole_2.2mm_M2, F.Cu at (53.5, 99.0)
Routing:
- net /processing/BLE_UART_TXD: track 29.6 -> 32.1 mm
- net Net-(U2-UART_RXD): track 25.4 -> 27.9 mm
Changed lines of the file:
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@@
 		)
 	)
+	(footprint "MountingHole:MountingHole_2.2mm_M2"
+		(layer "F.Cu")
+		(at 53.5 99.04)
+		(descr "Mounting Hole 2.2mm, M2, no annular, generated by kicad-footprint-generator mountinghole.py")
+		(tags "mountinghole M2")
+		(property "Reference" "REF**"
+			(at 0 -3.15 0)
+			(layer "F.SilkS")
+			(hide yes)
+			(effects
+				(font
+					(size 1 1)
+					(thickness 0.15)
+				)
+			)
+		)
+		(property "Value" "MountingHole_2.2mm_M2"
+			(at 0 3.15 0)
+			(layer "F.Fab")
+			(effects
+				(font
+					(size 1 1)
+					(thickness 0.15)
+				)
+			)
+		)
+		(property "Datasheet" ""
+			(at 0 0 0)
+			(layer "F.Fab")
+			(hide yes)
+			(effects
+				(font
+					(size 1.27 1.27)
+				)
+			)
+		)
+		(property "Description" ""
+			(at 0 0 0)
+			(layer "F.Fab")
+			(hide yes)
+			(effects
+				(font
+					(size 1.27 1.27)
+				)
+			)
+		)
+		(property "KiLib_Generator" "mounting_hardware/mounting_hole"
+			(at 0 0 0)
+			(layer "F.SilkS")
+			(hide yes)
+			(effects
+				(font
+					(size 1 1)
+					(thickness 0.15)
+				)
+			)
+		)
+		(attr exclude_from_pos_files exclude_from_bom)
+		(duplicate_pad_numbers_are_jumpers no)
+		(fp_circle
+			(center 0 0)
+			(end 2.2 0)
+			(stroke
+				(width 0.15)
+				(type solid)
+			)
+			(fill no)
+			(layer "Cmts.User")
+		)
+		(fp_circle
+			(center 0 0)
+			(end 2.45 0)
+			(stroke
+				(width 0.05)
+				(type solid)
+			)
+			(fill no)
+			(layer "F.CrtYd")
+		)
+		(fp_text user "${REFERENCE}"
+			(at 0 0 0)
+			(layer "F.Fab")
+			(effects
+				(font
+					(size 1 1)
+					(thickness 0.15)
+				)
+			)
+		)
+		(pad "" np_thru_hole circle
+			(at 0 0)
+			(size 2.2 2.2)
+			(drill 2.2)
+			(layers "*.Cu" "*.Mask")
+		)
+		(embedded_fonts no)
+	)
 	(footprint "easyeda2kicad:SW-SMD_4P-L6.2-W6.2-P4.00-LS6.8"
 		(layer "F.Cu")
@@
 	)
 	(segment
-		(start 39.68 107.05)
-		(end 41.51 108.88)
+		(start 52.337893 101.695)
+		(end 49.41 104.622892)
 		(width 0.15)
 		(layer "B.Cu")
@@
 	)
 	(segment
-		(start 52.337893 101.695)
-		(end 53.375 101.695)
+		(start 58.74 101.36)
+		(end 58.29 101.81)
 		(width 0.15)
 		(layer "B.Cu")
@@
 	(segment
 		(start 56.256446 100.86)
-		(end 57.206446 101.81)
+		(end 54.21 100.86)
 		(width 0.15)
 		(layer "B.Cu")
@@
 	)
 	(segment
-		(start 49.41 107.596446)
-		(end 49.41 104.622892)
+		(start 49.41 104.622892)
+		(end 49.41 107.596446)
 		(width 0.15)
 		(layer "B.Cu")
@@
 	)
 	(segment
-		(start 57.206446 101.81)
-		(end 58.29 101.81)
+		(start 49.41 107.596446)
+		(end 46.436446 110.57)
 		(width 0.15)
 		(layer "B.Cu")
@@
 	)
 	(segment
-		(start 39.68 105.86)
-		(end 39.68 107.05)
+		(start 61.064734 101.36)
+		(end 58.74 101.36)
 		(width 0.15)
 		(layer "B.Cu")
@@
 	)
 	(segment
-		(start 53.375 101.695)
-		(end 54.21 100.86)
+		(start 39.68 109.006446)
+		(end 39.68 105.86)
 		(width 0.15)
 		(layer "B.Cu")
@@
 	)
 	(segment
-		(start 58.74 101.36)
-		(end 61.064734 101.36)
+		(start 46.436446 110.57)
+		(end 41.243554 110.57)
 		(width 0.15)
 		(layer "B.Cu")
@@
 	)
 	(segment
-		(start 48.126446 108.88)
-		(end 49.41 107.596446)
+		(start 61.498719 101.793985)
+		(end 61.064734 101.36)
 		(width 0.15)
 		(layer "B.Cu")
@@
 	(segment
 		(start 58.29 101.81)
-		(end 58.74 101.36)
+		(end 57.206446 101.81)
 		(width 0.15)
 		(layer "B.Cu")
@@
 	)
 	(segment
-		(start 61.064734 101.36)
-		(end 61.498719 101.793985)
+		(start 57.206446 101.81)
+		(end 56.256446 100.86)
 		(width 0.15)
 		(layer "B.Cu")
@@
 	)
 	(segment
-		(start 54.21 100.86)
-		(end 56.256446 100.86)
+		(start 41.243554 110.57)
+		(end 39.68 109.006446)
 		(width 0.15)
 		(layer "B.Cu")
@@
 	)
 	(segment
-		(start 49.41 104.622892)
+		(start 53.375 101.695)
 		(end 52.337893 101.695)
 		(width 0.15)
@@
 	)
 	(segment
-		(start 41.51 108.88)
-		(end 48.126446 108.88)
+		(start 54.21 100.86)
+		(end 53.375 101.695)
 		(width 0.15)
 		(layer "B.Cu")
@@
 	)
 	(segment
-		(start 38.765001 103.120001)
-		(end 38.765001 106.555001)
+		(start 53.795 101.945)
+		(end 52.441446 101.945)
 		(width 0.15)
 		(layer "B.Cu")
@@
 	)
 	(segment
-		(start 41.34 109.13)
-		(end 48.23 109.13)
+		(start 52.441446 101.945)
+		(end 49.66 104.726446)
 		(width 0.15)
 		(layer "B.Cu")
@@
 	)
 	(segment
-		(start 53.795 101.945)
-		(end 54.16 101.58)
+		(start 46.54 110.82)
+		(end 41.14 110.82)
 		(width 0.15)
 		(layer "B.Cu")
@@
 	)
 	(segment
-		(start 52.441446 101.945)
-		(end 53.795 101.945)
+		(start 54.830001 101.58)
+		(end 54.16 101.58)
 		(width 0.15)
 		(layer "B.Cu")
@@
 	)
 	(segment
-		(start 49.66 107.7)
-		(end 49.66 104.726446)
+		(start 38.765001 108.445001)
+		(end 38.765001 103.120001)
 		(width 0.15)
 		(layer "B.Cu")
@@
 	(segment
 		(start 54.16 101.58)
-		(end 54.830001 101.58)
+		(end 53.795 101.945)
 		(width 0.15)
 		(layer "B.Cu")
@@
 	)
 	(segment
-		(start 48.23 109.13)
-		(end 49.66 107.7)
+		(start 49.66 107.7)
+		(end 46.54 110.82)
 		(width 0.15)
 		(layer "B.Cu")
@@
 	)
 	(segment
-		(start 38.765001 106.555001)
-		(end 41.34 109.13)
+		(start 41.14 110.82)
+		(end 38.765001 108.445001)
 		(width 0.15)
 		(layer "B.Cu")
@@
 	(segment
 		(start 49.66 104.726446)
-		(end 52.441446 101.945)
+		(end 49.66 107.7)
 		(width 0.15)
 		(layer "B.Cu")

Commit message: firmware/journal update
Parts:
- removed REF** (x3): MountingHole_2.2mm_M2, MountingHole:MountingHole_2.2mm_M2
- moved R8 1.22 mm to (64.8, 136.3), turned to -135 degrees
Connections:
- J1 pad 1: /processing/GPIO31 -> /processing/SD_DAT3
- J1 pad 2: /processing/GPIO27 -> /processing/SD_CMD
- J1 pad 5: /processing/GPIO26 -> /processing/SD_CLK
- J1 pad 7: /processing/GPIO28 -> /processing/SD_DAT0
- J1 pad 8: /processing/GPIO29 -> /processing/SD_DAT1
- J1 pad 9: /processing/GPIO30 -> /processing/SD_DAT2
- R10 pad 2: /processing/GPIO28 -> /processing/SD_DAT0
- R11 pad 2: /processing/GPIO29 -> /processing/SD_DAT1
- R7 pad 2: /processing/GPIO27 -> /processing/SD_CMD
- R8 pad 2: /processing/GPIO31 -> /processing/SD_DAT3
- R9 pad 2: /processing/GPIO30 -> /processing/SD_DAT2
- U6 pad 26: /processing/DB5 -> /processing/DB6
- U6 pad 27: /processing/DB6 -> /processing/DB7
- U6 pad 28: /processing/DB7 -> /processing/DB8
- U6 pad 36: /processing/DB8 -> /processing/DB9
- U6 pad 37: /processing/DB9 -> /processing/DB10
- U6 pad 38: /processing/DB10 -> /processing/DB11
- U6 pad 39: /processing/DB11 -> /processing/DB12
- U6 pad 40: /processing/DB12 -> /processing/DB13
- U6 pad 42: /processing/DB13 -> /processing/DB14
- U6 pad 43: /processing/DB14 -> /processing/DB15
- U6 pad 44: /processing/DB15 -> /processing/DB16
- U6 pad 45: /processing/DB16 -> /processing/DB17
- U6 pad 46: /processing/DB17 -> unconnected-(U6-GPIO37-Pad46)
- U6 pad 49: /processing/GPIO31 -> /processing/SD_CLK
- U6 pad 52: /processing/GPIO30 -> /processing/SD_CMD
- U6 pad 53: /processing/GPIO29 -> /processing/SD_DAT0
- U6 pad 54: /processing/GPIO28 -> /processing/SD_DAT1
- U6 pad 55: /processing/GPIO27 -> /processing/SD_DAT2
- U6 pad 56: /processing/GPIO26 -> /processing/SD_DAT3
Routing:
- net /processing/GPIO29: track 72.7 -> 0.00 mm
- net /processing/GPIO28: track 70.3 -> 0.00 mm
- net /processing/SD_DAT1: track 0.00 -> 67.6 mm
- net /processing/SD_DAT0: track 0.00 -> 66.5 mm
- net /processing/GPIO26: track 58.7 -> 0.00 mm
- net /processing/SD_CLK: track 0.00 -> 55.6 mm
- net /processing/GPIO27: track 52.9 -> 0.00 mm
- net /processing/SD_DAT3: track 0.00 -> 50.3 mm
- net /processing/SD_CMD: track 0.00 -> 49.7 mm
- net /processing/GPIO31: track 47.5 -> 0.00 mm
- net /processing/GPIO30: track 44.2 -> 0.00 mm
- net /processing/SD_DAT2: track 0.00 -> 42.4 mm
- net /processing/DB5: track 38.2 -> 0.00 mm
- net /processing/DB13: track 41.1 -> 38.6 mm
- net /processing/DB7: track 39.9 -> 38.9 mm
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