File: src/kicad/audio.kicad_sch (KiCad schematic)
At the start: 2 parts, among them J3 AudioJack4_SwitchTR1, U5 PCM5102A

Commit message: new journal entry!
Parts:
- added C26: 10uf, symbol Device:C
- added C39, C40: 2.2nf, symbol Device:C
- added C41, C42: 1uf, symbol Device:C
- added C43, C44, C46, C51: 0.1uf, symbol Device:C
- added C45, C48: 2.2uf, symbol Device:C
- added C47, C49, C50, C52: 10uf, symbol Device:C_Polarized
- added R22: 10k, symbol Device:R
- added R23, R24: 470, symbol Device:R
- added U10: LP5907MFX-3.3, Package_TO_SOT_SMD:SOT-23-5, symbol Regulator_Linear:LP5907MFX-3.3
Connections:
- net +3V3: now reaches U5.1 (CPVDD)
- net +3V3: now also U5.20 (DVDD), C42.1, C44.1, C50.1, C51.1, C52.2, U10.1 (IN)
- net GND: now reaches U5.10 (DEMP)
- net GND: now also J3.R2, J3.S, U5.11 (FLT), U5.16 (FMT), U5.19 (DGND), U5.3 (CPGND), U5.9 (AGND), C26.2, C39.1, C40.2, C41.2, C42.2, C43.2, C44.2, C46.1, C47.2, C48.1, C49.2, C50.2, C51.2, C52.1, U10.2 (GND)
- net I2S.SCK: now reaches U5.12 (SCK)
- net I2S.BCK: now reaches U5.13 (BCK)
- net I2S.DIN: now reaches U5.14 (DIN)
- net I2S.LRCK: now reaches U5.15 (LRCK)
- net at U5.17 (XSMT): now also C26.1, R22.2
- net at U5.18 (LDOO): now also C46.2, C47.1
- net at U5.2 (CAPP): now also C45.2
- net at U5.4 (CAPM): now also C45.1
- net at U5.5 (VNEG): now also C48.2
- net at U5.6 (OUTL): now also R23.1
- net at U5.7 (OUTR): now also R24.1
- net +3V3_ANALOG: now reaches U5.8 (AVDD)
- net +3V3_ANALOG: now also C41.1, C43.1, C49.1, R22.1, U10.5 (OUT)
- net RIGHT_AUDIO: now reaches J3.R1
- net RIGHT_AUDIO: now also C40.1, R24.2
- net LEFT_AUDIO: now reaches J3.T
- net LEFT_AUDIO: now also C39.2, R23.2
- net JACK_DETECTION: now reaches J3.TN
- new net ANALOG_LDO_EN: U10.3 (EN)
- no-connect marks 0 -> 1
Other:
- note added: "3.5mm jack port"
- note added: "check datasheet when routing please :rayge:"
- note added: "ldo for clean 3.3v for the analog circuit"
- moved on the sheet: J3, U5

Commit message: progress + new journal entry!
Parts:
- added R38, R39: 10k, symbol Device:R
Connections:
- net +3V3: now also R38.2
- net ANALOG_LDO_EN: now also R39.1
- net GND: now also R39.2
- net JACK_DETECTION: now also R38.1

Commit message: may 28th
Parts:
- R22, R38, R39: footprint (none) -> Resistor_SMD:R_0402_1005Metric
- R23, R24: footprint (none) -> Resistor_SMD:R_0603_1608Metric; LCSC Part (none) -> C218042; Tolerance (none) -> 1%
- U10: LCSC Part (none) -> C23380874
- U5: LCSC Part (none) -> C107671

Commit message: more components associations
Parts:
- R22, R38, R39: LCSC Part (none) -> C25744
Changed lines of the file:
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@@
+			)
+		)
+		(property "LCSC Part" "C25744"
+			(at 180.34 57.785 90)
+			(hide yes)
+			(show_name no)
+			(do_not_autoplace no)
+			(effects
+				(font
+					(size 1.27 1.27)
+				)
 			)
 		)
@@
 			)
 		)
+		(property "LCSC Part" "C25744"
+			(at 26.67 74.93 90)
+			(hide yes)
+			(show_name no)
+			(do_not_autoplace no)
+			(effects
+				(font
+					(size 1.27 1.27)
+				)
+			)
+		)
 		(pin "2"
 		)
@@
 			(at 39.37 129.54 0)
 			(hide yes)
+			(show_name no)
+			(do_not_autoplace no)
+			(effects
+				(font
+					(size 1.27 1.27)
+				)
+			)
+		)
+		(property "LCSC Part" "C25744"
+			(at 39.37 129.54 0)
+			(hide yes)

Commit message: may 29th + files updates
Parts:
- removed C47, C52: 10uf, symbol Device:C_Polarized
- removed J3: AudioJack4_SwitchTR1, symbol Connector_Audio:AudioJack4_SwitchTR1
- removed R38: 10k, Resistor_SMD:R_0402_1005Metric, symbol Device:R
- added C52, C57: 10uf, Capacitor_SMD:C_0805_2012Metric, symbol Device:C
- added C56: 100nf, Capacitor_SMD:C_0402_1005Metric, symbol Device:C
- added J7: AudioJack3_Ground_SwitchTR, easyeda2kicad:AUDIO-SMD_PJ-342-141, symbol Connector_Audio:AudioJack3_Ground_SwitchTR
- added Q4: BSS138, Package_TO_SOT_SMD:SOT-23, symbol Transistor_FET:BSS138
- added R30: 100k, Resistor_SMD:R_0402_1005Metric, symbol Device:R
- added R31: 10k, Resistor_SMD:R_0402_1005Metric, symbol Device:R
- C26, C49, C50: footprint (none) -> Capacitor_SMD:C_0603_1608Metric; LCSC Part (none) -> C96446
- C39, C40: footprint (none) -> Capacitor_SMD:C_0805_2012Metric; LCSC Part (none) -> C28260
- C41, C42: footprint (none) -> Capacitor_SMD:C_0402_1005Metric; LCSC Part (none) -> C52923
- C43, C44, C46, C51: footprint (none) -> Capacitor_SMD:C_0402_1005Metric; LCSC Part (none) -> C1525
- C45, C48: footprint (none) -> Capacitor_SMD:C_0402_1005Metric; LCSC Part (none) -> C12530
Connections:
- net +3V3: now also C52.2, R30.2, R31.2
- net GND: now also C52.1, C56.1, C57.2, J7.G, J7.S, Q4.2 (S)
- net JACK_DETECTION: now also Q4.3 (D), R31.1
- net LEFT_AUDIO: now also J7.T
- net RIGHT_AUDIO: now also J7.R
- net at C46.2, U5.18 (LDOO): now also C57.1
- new net SW_T: C56.2, J7.TN, Q4.1 (G), R30.1
Other:
- moved on the sheet: C26, C39, C40, C43, C44, C45, C46, C48, C49, C50, C51, R22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

Commit message: routing + may 30th update + things
Parts:
- C41: value 1uf -> 4.7uf; footprint Capacitor_SMD:C_0402_1005Metric -> Capacitor_SMD:C_0603_1608Metric; LCSC Part C52923 -> C19666
Changed lines of the file:
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@@
 	)
 	(label "SW_T"
-		(at 38.1 172.085 180)
+		(at 38.1 172.085 0)
 		(effects
 			(font
 				(size 1.27 1.27)
 			)
-			(justify right bottom)
+			(justify left bottom)
 		)
 	)
@@
 			)
 		)
-		(property "Value" "1uf"
+		(property "Value" "4.7uf"
 			(at 176.53 25.4 90)
 			(show_name no)
@@
 			)
 		)
-		(property "Footprint" "Capacitor_SMD:C_0402_1005Metric"
+		(property "Footprint" "Capacitor_SMD:C_0603_1608Metric"
 			(at 180.34 29.5148 0)
 			(hide yes)
@@
 			)
 		)
-		(property "LCSC Part" "C52923"
+		(property "LCSC Part" "C19666"
 			(at 176.53 30.48 90)
 			(hide yes)

Commit message: cad added + journal/bom update
Parts:
- C42: LCSC Part C52923 -> C307427
- C43, C44, C46, C51: value 0.1uf -> 100nf
- C52, C57: LCSC Part C15850 -> C1713
- R22, R31, R39: LCSC Part C25744 -> C2906861
- R30: LCSC Part C25741 -> C481918
Changed lines of the file:
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@@
 			)
 		)
-		(property "LCSC Part" "C25741"
+		(property "LCSC Part" "C481918"
 			(at 43.815 177.8 0)
 			(hide yes)
@@
 			)
 		)
-		(property "Value" "0.1uf"
+		(property "Value" "100nf"
 			(at 88.265 85.09 0)
 			(show_name no)
@@
 			)
 		)
-		(property "Value" "0.1uf"
+		(property "Value" "100nf"
 			(at 62.23 36.195 90)
 			(show_name no)
@@
 			)
 		)
-		(property "Value" "0.1uf"
+		(property "Value" "100nf"
 			(at 104.14 67.945 0)
 			(show_name no)
@@
 			)
 		)
-		(property "Value" "0.1uf"
+		(property "Value" "100nf"
 			(at 51.054 36.957 90)
 			(show_name no)
@@
 			)
 		)
-		(property "LCSC Part" "C25744"
+		(property "LCSC Part" "C2906861"
 			(at 180.34 57.785 90)
 			(hide yes)
@@
 			)
 		)
-		(property "LCSC Part" "C52923"
+		(property "LCSC Part" "C307427"
 			(at 168.91 60.96 90)
 			(hide yes)
@@
 			)
 		)
-		(property "LCSC Part" "C25744"
+		(property "LCSC Part" "C2906861"
 			(at 63.5 164.465 90)
 			(hide yes)
@@
 			)
 		)
-		(property "LCSC Part" "C15850"
+		(property "LCSC Part" "C1713"
 			(at 100.33 85.725 90)
 			(hide yes)
@@
 			)
 		)
-		(property "LCSC Part" "C15850"
+		(property "LCSC Part" "C1713"
 			(at 83.82 68.58 90)
 			(hide yes)
@@
 			)
 		)
-		(property "LCSC Part" "C25744"
+		(property "LCSC Part" "C2906861"
 			(at 24.13 71.755 90)
 			(hide yes)
